Commit message: Modified colour of link 5 from yellow to grey

File: staubli_rx160_gazebo/urdf/rx160_macro.xacro (robot description, xacro)
@@ -89,5 +89,5 @@
   </gazebo>
   <gazebo reference="${prefix}link_5">
-    <material>Gazebo/Yellow</material>
+    <material>Gazebo/Grey</material>
     <turnGravityOff>true</turnGravityOff>
   </gazebo>

File: staubli_rx160_gazebo/urdf/rx160l_macro.xacro (robot description, xacro)
@@ -89,5 +89,5 @@
   </gazebo>
   <gazebo reference="${prefix}link_5">
-    <material>Gazebo/Yellow</material>
+    <material>Gazebo/Grey</material>
     <turnGravityOff>true</turnGravityOff>
   </gazebo>
