Commit message: Updated gazebo packages for rx160, tx90 series and support packages for tx90 series

File: staubli_tx90_support/urdf/tx90l_macro.xacro (robot description, xacro)
@@ -1,7 +1,7 @@
 <?xml version="1.0"?>
-<robot xmlns:xacro="http://ros.org/wiki/xacro">
+<robot xmlns:xacro="http://wiki.ros.org/xacro">
   <xacro:include filename="$(find staubli_resources)/urdf/common_materials.xacro"/>
   <xacro:macro name="staubli_tx90l" params="prefix">
-    <!-- links -->
+    <!-- links: main serial chain -->
     <link name="${prefix}base_link">
       <visual>
@@ -158,6 +158,5 @@
       </inertial>
     </link>
-    <link name="${prefix}tool0"/>
-    <!-- joints -->
+    <!-- joints: main serial chain -->
     <joint name="${prefix}joint_1" type="revolute">
       <origin xyz="0 0 0.478" rpy="0 0 0"/>
@@ -168,5 +167,5 @@
       (1) effort limit = 318 Nm if floor mounted
       (2) effort limit = 111 Nm if wall mounted -->
-      <limit lower="-3.14159" upper="3.14159" effort="318.0" velocity="3.75" />
+      <limit lower="${radians(-180)}" upper="${radians(180)}" effort="318.0" velocity="${radians(400)}" />
       <dynamics damping="0.0" friction="0.0"/>
     </joint>
@@ -176,5 +175,5 @@
       <child link="${prefix}link_2"/>
       <axis xyz="0 1 0"/>
-      <limit lower="-2.268928" upper="2.574360" effort="130.0" velocity="2.97" />
+      <limit lower="${radians(-130)}" upper="${radians(147.5)}" effort="130.0" velocity="${radians(390)}" />
       <dynamics damping="0.0" friction="0.0"/>
     </joint>
@@ -184,5 +183,5 @@
       <child link="${prefix}link_3"/>
       <axis xyz="0 1 0"/>
-      <limit lower="-2.530727" upper="2.530727" effort="65.0" velocity="4.45" />
+      <limit lower="${radians(-145)}" upper="${radians(145)}" effort="65.0" velocity="${radians(420)}" />
       <dynamics damping="0.0" friction="0.0"/>
     </joint>
@@ -192,5 +191,5 @@
       <child link="${prefix}link_4"/>
       <axis xyz="0 0 1"/>
-      <limit lower="-4.712389" upper="4.712389" effort="34.0" velocity="7.50" />
+      <limit lower="${radians(-270)}" upper="${radians(270)}" effort="34.0" velocity="${radians(540)}" />
       <dynamics damping="0.0" friction="0.0"/>
     </joint>
@@ -200,5 +199,5 @@
       <child link="${prefix}link_5"/>
       <axis xyz="0 1 0"/>
-      <limit lower="-2.007129" upper="2.443461" effort="29.0" velocity="6.11" />
+      <limit lower="${radians(-115)}" upper="${radians(140)}" effort="29.0" velocity="${radians(475)}" />
       <dynamics damping="0.0" friction="0.0"/>
     </joint>
@@ -208,5 +207,5 @@
       <child link="${prefix}link_6"/>
       <axis xyz="0 0 1"/>
-      <limit lower="-4.712389" upper="4.712389" effort="11.0" velocity="10.47" />
+      <limit lower="${radians(-270)}" upper="${radians(270)}" effort="11.0" velocity="${radians(760)}" />
       <dynamics damping="0.0" friction="0.0"/>
     </joint>
@@ -216,4 +215,25 @@
       <origin xyz="0 0 0" rpy="0 0 0"/>
     </joint>
+    <!-- ROS-Industrial 'base' frame: base_link to Staubli World Coordinates transform -->
+    <link name="${prefix}base" />
+    <joint name="${prefix}base_link-base" type="fixed">
+      <origin xyz="0 0 0.478" rpy="0 0 0"/>
+      <parent link="${prefix}base_link"/>
+      <child link="${prefix}base"/>
+    </joint>
+    <!-- ROS-Industrial 'flange' frame: attachment point for EEF models -->
+    <link name="${prefix}flange" />
+    <joint name="${prefix}joint_6-flange" type="fixed">
+      <origin xyz="0 0 0" rpy="0 ${radians(-90.0)} 0" />
+      <parent link="${prefix}link_6" />
+      <child link="${prefix}flange" />
+    </joint>
+    <!-- ROS-Industrial 'tool0' frame: all-zeros tool frame -->
+    <link name="${prefix}tool0" />
+    <joint name="${prefix}flange-tool0" type="fixed">
+      <origin xyz="0 0 0" rpy="0 ${radians(90.0)} 0" />
+      <parent link="${prefix}flange" />
+      <child link="${prefix}tool0" />
+    </joint>
   </xacro:macro>
 </robot>

File: staubli_tx90_support/urdf/tx90xl.xacro (robot description, xacro)
@@ -1,4 +1,4 @@
 <?xml version="1.0" ?>
-<robot name="staubli_tx90xl" xmlns:xacro="http://ros.org/wiki/xacro">
+<robot name="staubli_tx90xl" xmlns:xacro="http://wiki.ros.org/xacro">
   <xacro:include filename="$(find staubli_tx90_support)/urdf/tx90xl_macro.xacro"/>
   <xacro:staubli_tx90xl prefix=""/>

File: staubli_tx90_support/urdf/tx90xl_macro.xacro (robot description, xacro)
@@ -1,7 +1,7 @@
 <?xml version="1.0"?>
-<robot xmlns:xacro="http://ros.org/wiki/xacro">
+<robot xmlns:xacro="http://wiki.ros.org/xacro">
   <xacro:include filename="$(find staubli_resources)/urdf/common_materials.xacro"/>
   <xacro:macro name="staubli_tx90xl" params="prefix">
-    <!-- links -->
+    <!-- links: main serial chain -->
     <link name="${prefix}base_link">
       <visual>
@@ -158,6 +158,5 @@
       </inertial>
     </link>
-    <link name="${prefix}tool0"/>
-    <!-- joints -->
+    <!-- joints: main serial chain -->
     <joint name="${prefix}joint_1" type="revolute">
       <origin xyz="0 0 0.478" rpy="0 0 0"/>
@@ -168,5 +167,5 @@
       (1) effort limit = 318 Nm if floor mounted
       (2) effort limit = 111 Nm if wall mounted -->
-      <limit lower="-3.14159" upper="3.14159" effort="318.0" velocity="3.32" />
+      <limit lower="${radians(-180)}" upper="${radians(180)}" effort="318.0" velocity="${radians(400)}" />
       <dynamics damping="0.0" friction="0.0"/>
     </joint>
@@ -176,5 +175,5 @@
       <child link="${prefix}link_2"/>
       <axis xyz="0 1 0"/>
-      <limit lower="-2.268928" upper="2.574360" effort="90.0" velocity="2.79" />
+      <limit lower="${radians(-130)}" upper="${radians(147.5)}" effort="90.0" velocity="${radians(350)}" />
       <dynamics damping="0.0" friction="0.0"/>
     </joint>
@@ -184,5 +183,5 @@
       <child link="${prefix}link_3"/>
       <axis xyz="0 1 0"/>
-      <limit lower="-2.530727" upper="2.530727" effort="53.0" velocity="4.01" />
+      <limit lower="${radians(-145)}" upper="${radians(145)}" effort="53.0" velocity="${radians(410)}" />
       <dynamics damping="0.0" friction="0.0"/>
     </joint>
@@ -192,5 +191,5 @@
       <child link="${prefix}link_4"/>
       <axis xyz="0 0 1"/>
-      <limit lower="-4.712389" upper="4.712389" effort="34.0" velocity="6.98" />
+      <limit lower="${radians(-270)}" upper="${radians(270)}" effort="34.0" velocity="${radians(540)}" />
       <dynamics damping="0.0" friction="0.0"/>
     </joint>
@@ -200,5 +199,5 @@
       <child link="${prefix}link_5"/>
       <axis xyz="0 1 0"/>
-      <limit lower="-2.007129" upper="2.443461" effort="29.0" velocity="6.02" />
+      <limit lower="${radians(-115)}" upper="${radians(140)}" effort="29.0" velocity="${radians(475)}" />
       <dynamics damping="0.0" friction="0.0"/>
     </joint>
@@ -208,5 +207,5 @@
       <child link="${prefix}link_6"/>
       <axis xyz="0 0 1"/>
-      <limit lower="-4.712389" upper="4.712389" effort="11.0" velocity="10.47" />
+      <limit lower="${radians(-270)}" upper="${radians(270)}" effort="11.0" velocity="${radians(760)}" />
       <dynamics damping="0.0" friction="0.0"/>
     </joint>
@@ -216,4 +215,25 @@
       <origin xyz="0 0 0" rpy="0 0 0"/>
     </joint>
+    <!-- ROS-Industrial 'base' frame: base_link to Staubli World Coordinates transform -->
+    <link name="${prefix}base" />
+    <joint name="${prefix}base_link-base" type="fixed">
+      <origin xyz="0 0 0.478" rpy="0 0 0"/>
+      <parent link="${prefix}base_link"/>
+      <child link="${prefix}base"/>
+    </joint>
+    <!-- ROS-Industrial 'flange' frame: attachment point for EEF models -->
+    <link name="${prefix}flange" />
+    <joint name="${prefix}joint_6-flange" type="fixed">
+      <origin xyz="0 0 0" rpy="0 ${radians(-90.0)} 0" />
+      <parent link="${prefix}link_6" />
+      <child link="${prefix}flange" />
+    </joint>
+    <!-- ROS-Industrial 'tool0' frame: all-zeros tool frame -->
+    <link name="${prefix}tool0" />
+    <joint name="${prefix}flange-tool0" type="fixed">
+      <origin xyz="0 0 0" rpy="0 ${radians(90.0)} 0" />
+      <parent link="${prefix}flange" />
+      <child link="${prefix}tool0" />
+    </joint>
   </xacro:macro>
 </robot>
