Commit message: Using common meshes across robots where possible

File: staubli_tx90_support/urdf/tx90l.urdf (robot description, URDF)
Before this commit: robot staubli_tx90, 8 links, 7 joints
Links:
- link link_2: mass 12.98711 -> 14.350897; geometry collision mesh filename=package://staubli_tx90_support/meshes/tx90l/collision/link_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; visual mesh filename=package://staubli_tx90_support/meshes/tx90l/visual/link_2.s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
- link link_3: mass 7.50151 -> 7.501506
- link link_4: mass 4.54015 -> 6.420429; geometry collision mesh filename=package://staubli_tx90_support/meshes/tx90l/collision/link_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; visual mesh filename=package://staubli_tx90_support/meshes/tx90l/visual/link_4.s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
- link link_5: mass 0.56876 -> 0.568760
- link link_6: mass 0.03098 -> 0.030977
Joints:
- joint joint_1: limit lower=-3.141593 upper=3.141593 effort=318.0 velocity=4.36 -> lower=-3.14159 upper=3.14159 effort=318.0 velocity=3.75
- joint joint_2: limit lower=-2.268928 upper=2.574360 effort=166.0 velocity=3.49 -> lower=-2.268928 upper=2.574360 effort=130.0 velocity=2.97
- joint joint_3: limit lower=-2.530727 upper=2.530727 effort=76.0 velocity=5.24 -> lower=-2.530727 upper=2.530727 effort=65.0 velocity=4.45; origin xyz=0 0.05 0.425 rpy=0 0 0 -> xyz=0 0.05 0.500 rpy=0 0 0
- joint joint_5: origin xyz=0 0 0.425 rpy=0 0 0 -> xyz=0 0 0.550 rpy=0 0 0

File: staubli_tx90_support/urdf/tx90l_macro.xacro (robot description, xacro)
@@ -8,12 +8,12 @@
         <origin xyz="0 0 0" rpy="0 0 0"/>
         <geometry>
-          <mesh filename="package://staubli_tx90_support/meshes/tx90l/visual/base_link.stl"/>
-        </geometry>
-        <xacro:material_staubli_ral_melon_yellow />
-      </visual>
-      <collision>
-        <origin xyz="0 0 0" rpy="0 0 0"/>
-        <geometry>
-          <mesh filename="package://staubli_tx90_support/meshes/tx90l/collision/base_link.stl"/>
+          <mesh filename="package://staubli_tx90_support/meshes/tx90/visual/base_link.stl"/>
+        </geometry>
+        <xacro:material_staubli_ral_melon_yellow />
+      </visual>
+      <collision>
+        <origin xyz="0 0 0" rpy="0 0 0"/>
+        <geometry>
+          <mesh filename="package://staubli_tx90_support/meshes/tx90/collision/base_link.stl"/>
         </geometry>
       </collision>
@@ -30,12 +30,12 @@
         <origin xyz="0 0 0" rpy="0 0 0"/>
         <geometry>
-          <mesh filename="package://staubli_tx90_support/meshes/tx90l/visual/link_1.stl"/>
-        </geometry>
-        <xacro:material_staubli_ral_melon_yellow />
-      </visual>
-      <collision>
-        <origin xyz="0 0 0" rpy="0 0 0"/>
-        <geometry>
-          <mesh filename="package://staubli_tx90_support/meshes/tx90l/collision/link_1.stl"/>
+          <mesh filename="package://staubli_tx90_support/meshes/tx90/visual/link_1.stl"/>
+        </geometry>
+        <xacro:material_staubli_ral_melon_yellow />
+      </visual>
+      <collision>
+        <origin xyz="0 0 0" rpy="0 0 0"/>
+        <geometry>
+          <mesh filename="package://staubli_tx90_support/meshes/tx90/collision/link_1.stl"/>
         </geometry>
       </collision>
@@ -74,12 +74,12 @@
         <origin xyz="0 0 0" rpy="0 0 0"/>
         <geometry>
-          <mesh filename="package://staubli_tx90_support/meshes/tx90l/visual/link_3.stl"/>
-        </geometry>
-        <xacro:material_staubli_ral_melon_yellow />
-      </visual>
-      <collision>
-        <origin xyz="0 0 0" rpy="0 0 0"/>
-        <geometry>
-          <mesh filename="package://staubli_tx90_support/meshes/tx90l/collision/link_3.stl"/>
+          <mesh filename="package://staubli_tx90_support/meshes/tx90/visual/link_3.stl"/>
+        </geometry>
+        <xacro:material_staubli_ral_melon_yellow />
+      </visual>
+      <collision>
+        <origin xyz="0 0 0" rpy="0 0 0"/>
+        <geometry>
+          <mesh filename="package://staubli_tx90_support/meshes/tx90/collision/link_3.stl"/>
         </geometry>
       </collision>
@@ -118,5 +118,5 @@
         <origin xyz="0 0 0" rpy="0 0 0"/>
         <geometry>
-          <mesh filename="package://staubli_tx90_support/meshes/tx90l/visual/link_5.stl"/>
+          <mesh filename="package://staubli_tx90_support/meshes/tx90/visual/link_5.stl"/>
         </geometry>
         <xacro:material_staubli_ral_grey_aluminium />
@@ -125,5 +125,5 @@
         <origin xyz="0 0 0" rpy="0 0 0"/>
         <geometry>
-          <mesh filename="package://staubli_tx90_support/meshes/tx90l/collision/link_5.stl"/>
+          <mesh filename="package://staubli_tx90_support/meshes/tx90/collision/link_5.stl"/>
         </geometry>
       </collision>
@@ -140,5 +140,5 @@
         <origin xyz="0 0 0" rpy="0 0 0"/>
         <geometry>
-          <mesh filename="package://staubli_tx90_support/meshes/tx90l/visual/link_6.stl"/>
+          <mesh filename="package://staubli_tx90_support/meshes/tx90/visual/link_6.stl"/>
         </geometry>
         <xacro:material_staubli_ral_grey_aluminium />
@@ -147,5 +147,5 @@
         <origin xyz="0 0 0" rpy="0 0 0"/>
         <geometry>
-          <mesh filename="package://staubli_tx90_support/meshes/tx90l/collision/link_6.stl"/>
+          <mesh filename="package://staubli_tx90_support/meshes/tx90/collision/link_6.stl"/>
         </geometry>
       </collision>

File: staubli_tx90_support/urdf/tx90xl.urdf (robot description, URDF)
Before this commit: robot staubli_tx90, 8 links, 7 joints
Links:
- link link_2: mass 12.98711 -> 17.789372; geometry collision mesh filename=package://staubli_tx90_support/meshes/tx90xl/collision/link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; visual mesh filename=package://staubli_tx90_support/meshes/tx90xl/visual/link_2.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
- link link_3: mass 7.50151 -> 7.501506
- link link_4: mass 4.54015 -> 7.916800; geometry collision mesh filename=package://staubli_tx90_support/meshes/tx90xl/collision/link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; visual mesh filename=package://staubli_tx90_support/meshes/tx90xl/visual/link_4.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
- link link_5: mass 0.56876 -> 0.568760
- link link_6: mass 0.03098 -> 0.030977
Joints:
- joint joint_1: limit lower=-3.141593 upper=3.141593 effort=318.0 velocity=4.36 -> lower=-3.14159 upper=3.14159 effort=318.0 velocity=3.32
- joint joint_2: limit lower=-2.268928 upper=2.574360 effort=166.0 velocity=3.49 -> lower=-2.268928 upper=2.574360 effort=90.0 velocity=2.79
- joint joint_3: limit lower=-2.530727 upper=2.530727 effort=76.0 velocity=5.24 -> lower=-2.530727 upper=2.530727 effort=53.0 velocity=4.01; origin xyz=0 0.05 0.425 rpy=0 0 0 -> xyz=0 0.05 0.650 rpy=0 0 0
- joint joint_4: limit lower=-4.712389 upper=4.712389 effort=34.0 velocity=7.50 -> lower=-4.712389 upper=4.712389 effort=34.0 velocity=6.98
- joint joint_5: limit lower=-2.007129 upper=2.443461 effort=29.0 velocity=6.11 -> lower=-2.007129 upper=2.443461 effort=29.0 velocity=6.02; origin xyz=0 0 0.425 rpy=0 0 0 -> xyz=0 0 0.650 rpy=0 0 0

File: staubli_tx90_support/urdf/tx90xl_macro.xacro (robot description, xacro)
@@ -8,12 +8,12 @@
         <origin xyz="0 0 0" rpy="0 0 0"/>
         <geometry>
-          <mesh filename="package://staubli_tx90_support/meshes/tx90xl/visual/base_link.stl"/>
-        </geometry>
-        <xacro:material_staubli_ral_melon_yellow />
-      </visual>
-      <collision>
-        <origin xyz="0 0 0" rpy="0 0 0"/>
-        <geometry>
-          <mesh filename="package://staubli_tx90_support/meshes/tx90xl/collision/base_link.stl"/>
+          <mesh filename="package://staubli_tx90_support/meshes/tx90/visual/base_link.stl"/>
+        </geometry>
+        <xacro:material_staubli_ral_melon_yellow />
+      </visual>
+      <collision>
+        <origin xyz="0 0 0" rpy="0 0 0"/>
+        <geometry>
+          <mesh filename="package://staubli_tx90_support/meshes/tx90/collision/base_link.stl"/>
         </geometry>
       </collision>
@@ -30,12 +30,12 @@
         <origin xyz="0 0 0" rpy="0 0 0"/>
         <geometry>
-          <mesh filename="package://staubli_tx90_support/meshes/tx90xl/visual/link_1.stl"/>
-        </geometry>
-        <xacro:material_staubli_ral_melon_yellow />
-      </visual>
-      <collision>
-        <origin xyz="0 0 0" rpy="0 0 0"/>
-        <geometry>
-          <mesh filename="package://staubli_tx90_support/meshes/tx90xl/collision/link_1.stl"/>
+          <mesh filename="package://staubli_tx90_support/meshes/tx90/visual/link_1.stl"/>
+        </geometry>
+        <xacro:material_staubli_ral_melon_yellow />
+      </visual>
+      <collision>
+        <origin xyz="0 0 0" rpy="0 0 0"/>
+        <geometry>
+          <mesh filename="package://staubli_tx90_support/meshes/tx90/collision/link_1.stl"/>
         </geometry>
       </collision>
@@ -74,12 +74,12 @@
         <origin xyz="0 0 0" rpy="0 0 0"/>
         <geometry>
-          <mesh filename="package://staubli_tx90_support/meshes/tx90xl/visual/link_3.stl"/>
-        </geometry>
-        <xacro:material_staubli_ral_melon_yellow />
-      </visual>
-      <collision>
-        <origin xyz="0 0 0" rpy="0 0 0"/>
-        <geometry>
-          <mesh filename="package://staubli_tx90_support/meshes/tx90xl/collision/link_3.stl"/>
+          <mesh filename="package://staubli_tx90_support/meshes/tx90/visual/link_3.stl"/>
+        </geometry>
+        <xacro:material_staubli_ral_melon_yellow />
+      </visual>
+      <collision>
+        <origin xyz="0 0 0" rpy="0 0 0"/>
+        <geometry>
+          <mesh filename="package://staubli_tx90_support/meshes/tx90/collision/link_3.stl"/>
         </geometry>
       </collision>
@@ -118,5 +118,5 @@
         <origin xyz="0 0 0" rpy="0 0 0"/>
         <geometry>
-          <mesh filename="package://staubli_tx90_support/meshes/tx90xl/visual/link_5.stl"/>
+          <mesh filename="package://staubli_tx90_support/meshes/tx90/visual/link_5.stl"/>
         </geometry>
         <xacro:material_staubli_ral_grey_aluminium />
@@ -125,5 +125,5 @@
         <origin xyz="0 0 0" rpy="0 0 0"/>
         <geometry>
-          <mesh filename="package://staubli_tx90_support/meshes/tx90xl/collision/link_5.stl"/>
+          <mesh filename="package://staubli_tx90_support/meshes/tx90/collision/link_5.stl"/>
         </geometry>
       </collision>
@@ -140,5 +140,5 @@
         <origin xyz="0 0 0" rpy="0 0 0"/>
         <geometry>
-          <mesh filename="package://staubli_tx90_support/meshes/tx90xl/visual/link_6.stl"/>
+          <mesh filename="package://staubli_tx90_support/meshes/tx90/visual/link_6.stl"/>
         </geometry>
         <xacro:material_staubli_ral_grey_aluminium />
@@ -147,5 +147,5 @@
         <origin xyz="0 0 0" rpy="0 0 0"/>
         <geometry>
-          <mesh filename="package://staubli_tx90_support/meshes/tx90xl/collision/link_6.stl"/>
+          <mesh filename="package://staubli_tx90_support/meshes/tx90/collision/link_6.stl"/>
         </geometry>
       </collision>
