Commit message: remove joint6->tool0
as there is also joint6->flange->tool0

File: staubli_tx90_support/urdf/tx90_macro.xacro (robot description, xacro)
@@ -210,9 +210,4 @@
       <dynamics damping="0.0" friction="0.0"/>
     </joint>
-    <joint name="${prefix}joint_6-tool0" type="fixed">
-      <parent link="${prefix}link_6"/>
-      <child link="${prefix}tool0"/>
-      <origin xyz="0 0 0" rpy="0 0 0"/>
-    </joint>
     <!-- ROS-Industrial 'base' frame: base_link to Staubli World Coordinates transform -->
     <link name="${prefix}base" />

File: staubli_tx90_support/urdf/tx90l_macro.xacro (robot description, xacro)
@@ -210,9 +210,4 @@
       <dynamics damping="0.0" friction="0.0"/>
     </joint>
-    <joint name="${prefix}joint_6-tool0" type="fixed">
-      <parent link="${prefix}link_6"/>
-      <child link="${prefix}tool0"/>
-      <origin xyz="0 0 0" rpy="0 0 0"/>
-    </joint>
     <!-- ROS-Industrial 'base' frame: base_link to Staubli World Coordinates transform -->
     <link name="${prefix}base" />

File: staubli_tx90_support/urdf/tx90xl_macro.xacro (robot description, xacro)
@@ -210,9 +210,4 @@
       <dynamics damping="0.0" friction="0.0"/>
     </joint>
-    <joint name="${prefix}joint_6-tool0" type="fixed">
-      <parent link="${prefix}link_6"/>
-      <child link="${prefix}tool0"/>
-      <origin xyz="0 0 0" rpy="0 0 0"/>
-    </joint>
     <!-- ROS-Industrial 'base' frame: base_link to Staubli World Coordinates transform -->
     <link name="${prefix}base" />
