Commit message: Added STL-files and dimensions for the tx60l
TODO: jusitfy the frames for base and flange

File: staubli_tx60_support/urdf/tx60l_macro.xacro (robot description, xacro)
@@ -111,5 +111,5 @@
     <!-- joints: main serial chain -->
     <joint name="${prefix}joint_1" type="revolute">
-      <origin xyz="0 0 0.478" rpy="0 0 0"/>
+      <origin xyz="0 0 0.375" rpy="0 0 0"/>
       <parent link="${prefix}base_link"/>
       <child link="${prefix}link_1"/>
@@ -122,5 +122,5 @@
     </joint>
     <joint name="${prefix}joint_2" type="revolute">
-      <origin xyz="0.050 0 0" rpy="0 0 0"/>
+      <origin xyz="0 0 0" rpy="0 0 0"/>
       <parent link="${prefix}link_1"/>
       <child link="${prefix}link_2"/>
@@ -130,5 +130,5 @@
     </joint>
     <joint name="${prefix}joint_3" type="revolute">
-      <origin xyz="0 0.05 0.425" rpy="0 0 0"/>
+      <origin xyz="0 0.02 0.40" rpy="0 0 0"/>
       <parent link="${prefix}link_2"/>
       <child link="${prefix}link_3"/>
@@ -146,5 +146,5 @@
     </joint>
     <joint name="${prefix}joint_5" type="revolute">
-      <origin xyz="0 0 0.425" rpy="0 0 0"/>
+      <origin xyz="0 0 0.45" rpy="0 0 0"/>
       <parent link="${prefix}link_4"/>
       <child link="${prefix}link_5"/>
@@ -154,5 +154,5 @@
     </joint>
     <joint name="${prefix}joint_6" type="revolute">
-      <origin xyz="0 0 0.100" rpy="0 0 0"/>
+      <origin xyz="0 0 0.07" rpy="0 0 0"/>
       <parent link="${prefix}link_5"/>
       <child link="${prefix}link_6"/>

Commit message: added inertia matrices and masses for tx60l

File: staubli_tx60_support/urdf/tx60l_macro.xacro (robot description, xacro)
@@ -18,4 +18,11 @@
         </geometry>
       </collision>
+      <inertial>
+          <mass value="4.65971957"/>
+          <origin xyz="-0.00257355 -0.00039402 0.08786146" rpy="0.0 0.0 0.0"/>
+          <inertia ixx="0.02319781" ixy="0.00023234" ixz="0.00162421"
+                                    iyy="0.02621322" iyz="0.00008092"
+                                                     izz="0.02286303"/>
+      </inertial>
     </link>
     <link name="${prefix}link_1">
@@ -33,4 +40,11 @@
         </geometry>
       </collision>
+      <inertial>
+          <mass value="6.99103376"/>
+          <origin xyz="0.00000000 0.02467680 -0.05265925" rpy="0.0 0.0 0.0"/>
+          <inertia ixx="0.05672953" ixy="0.00000037" ixz="-0.00000049"
+                                    iyy="0.04909238" iyz="0.01016069"
+                                                     izz="0.03457565"/>
+      </inertial>
     </link>
     <link name="${prefix}link_2">
@@ -48,4 +62,11 @@
         </geometry>
       </collision>
+      <inertial>
+          <mass value="5.21353000"/>
+          <origin xyz="-0.00000322 0.17137541 0.17514843" rpy="0.0 0.0 0.0"/>
+          <inertia ixx="0.13669961" ixy="0.00000038" ixz="-0.00000068"
+                                    iyy="0.14393633" iyz="-0.00049262"
+                                                     izz="0.01130291"/>
+      </inertial>
     </link>
     <link name="${prefix}link_3">
@@ -63,4 +84,11 @@
         </geometry>
       </collision>
+      <inertial>
+          <mass value="4.52768000"/>
+          <origin xyz="0.00424668 0.02553862 -0.00735408" rpy="0.0 0.0 0.0"/>
+          <inertia ixx="0.02469218" ixy="0.00032528" ixz="0.00063194"
+                                    iyy="0.02222651" iyz="-0.00155762"
+                                                     izz="0.01657366"/>
+      </inertial>
     </link>
     <link name="${prefix}link_4">
@@ -78,4 +106,11 @@
         </geometry>
       </collision>
+      <inertial>
+          <mass value="3.48055000"/>
+          <origin xyz="-0.00134244 -0.00000186 0.28816464" rpy="0.0 0.0 0.0"/>
+          <inertia ixx="0.03950054" ixy="0.00000004" ixz="-0.00063419"
+                                    iyy="0.03813828" iyz="-0.00000002"
+                                                     izz="0.00610289"/>
+      </inertial>
     </link>
     <link name="${prefix}link_5">
@@ -93,4 +128,11 @@
         </geometry>
       </collision>
+      <inertial>
+          <mass value="0.16254714"/>
+          <origin xyz="-0.00000105 0.00000000 0.01268974" rpy="0.0 0.0 0.0"/>
+          <inertia ixx="0.00012557" ixy="0.00000000" ixz="0.00000000"
+                                    iyy="0.00013289" iyz="0.00000000"
+                                                     izz="0.00006342"/>
+      </inertial>
     </link>
     <link name="${prefix}link_6">
@@ -108,4 +150,11 @@
         </geometry>
       </collision>
+      <inertial>
+          <mass value="0.00820000"/>
+          <origin xyz="-0.00022629 0.00000000 -0.00597808" rpy="0.0 0.0 0.0"/>
+          <inertia ixx="0.00000096" ixy="0.00000000" ixz="0.00000000"
+                                    iyy="0.00000093" iyz="0.00000000"
+                                                     izz="0.00000154"/>
+      </inertial>
     </link>
     <!-- joints: main serial chain -->
