Commit message: Added STL-files for tx60

File: staubli_tx60_support/urdf/tx60_macro.xacro (robot description, xacro)
@@ -109,5 +109,4 @@
       </collision>
     </link>
-<!--LATER <link name="${prefix}tool0"/>-->
     <!-- joints: main serial chain -->
     <joint name="${prefix}joint_1" type="revolute">
@@ -162,8 +161,24 @@
       <dynamics damping="0.0" friction="0.0"/>
     </joint>
-    <joint name="${prefix}joint_6-tool0" type="fixed">
-      <parent link="${prefix}link_6"/>
-      <child link="${prefix}tool0"/>
-      <origin xyz="0 0 0" rpy="0 0 0"/>
+    <!-- ROS-Industrial 'base' frame: base_link to Fanuc World Coordinates transform -->
+    <link name="${prefix}base" />
+    <joint name="${prefix}base_link-base" type="fixed">
+      <origin xyz="0 0 0.650" rpy="0 0 0"/>
+      <parent link="${prefix}base_link"/>
+      <child link="${prefix}base"/>
+    </joint>
+    <!-- ROS-Industrial 'flange' frame: attachment point for EEF models -->
+    <link name="${prefix}flange" />
+    <joint name="${prefix}joint_6-flange" type="fixed">
+      <origin xyz="0 0 0" rpy="0 0 0" />
+      <parent link="${prefix}link_6" />
+      <child link="${prefix}flange" />
+    </joint>
+    <!-- ROS-Industrial 'tool0' frame: all-zeros tool frame -->
+    <link name="${prefix}tool0" />
+    <joint name="${prefix}link_6-tool0" type="fixed">
+      <origin xyz="0 0 0" rpy="0 0 0" />
+      <parent link="${prefix}link_6" />
+      <child link="${prefix}tool0" />
     </joint>
   </xacro:macro>

File: staubli_tx60_support/urdf/tx60l_macro.xacro (robot description, xacro)
@@ -3,10 +3,10 @@
   <xacro:include filename="$(find staubli_resources)/urdf/common_materials.xacro"/>
   <xacro:macro name="staubli_tx60l" params="prefix">
-    <!-- links -->
+    <!-- links: main serial chain -->
     <link name="${prefix}base_link">
       <visual>
         <origin xyz="0 0 0" rpy="0 0 0"/>
         <geometry>
-          <mesh filename="package://staubli_tx60_support/meshes/tx60/visual/base_link.stl"/>
+          <mesh filename="package://staubli_tx60_support/meshes/tx60l/visual/base_link.stl"/>
         </geometry>
         <xacro:material_staubli_ral_melon_yellow />
@@ -15,14 +15,7 @@
         <origin xyz="0 0 0" rpy="0 0 0"/>
         <geometry>
-          <mesh filename="package://staubli_tx60_support/meshes/tx60/collision/base_link.stl"/>
+          <mesh filename="package://staubli_tx60_support/meshes/tx60l/collision/base_link.stl"/>
         </geometry>
       </collision>
-      <inertial>
-          <mass value="10.733459"/>
-          <origin xyz="0.014288 0.000001 0.122264" rpy="0.0 0.0 0.0"/>
-          <inertia ixx="0.096560" ixy="-0.000005" ixz="-0.003803"
-                                  iyy="0.087591"  iyz="-0.000001"
-                                                  izz="0.081632"/>
-      </inertial>
     </link>
     <link name="${prefix}link_1">
@@ -30,5 +23,5 @@
         <origin xyz="0 0 0" rpy="0 0 0"/>
         <geometry>
-          <mesh filename="package://staubli_tx60_support/meshes/tx60/visual/link_1.stl"/>
+          <mesh filename="package://staubli_tx60_support/meshes/tx60l/visual/link_1.stl"/>
         </geometry>
         <xacro:material_staubli_ral_melon_yellow />
@@ -37,14 +30,7 @@
         <origin xyz="0 0 0" rpy="0 0 0"/>
         <geometry>
-          <mesh filename="package://staubli_tx60_support/meshes/tx60/collision/link_1.stl"/>
+          <mesh filename="package://staubli_tx60_support/meshes/tx60l/collision/link_1.stl"/>
         </geometry>
       </collision>
-      <inertial>
-          <mass value="16.934564"/>
-          <origin xyz="0.019143 0.024764 -0.064596" rpy="0.0 0.0 0.0"/>
-          <inertia ixx="0.222318" ixy="0.016499" ixz="0.023794"
-                                  iyy="0.208959" iyz="0.031663"
-                                                 izz="0.157081"/>
-      </inertial>
     </link>
     <link name="${prefix}link_2">
@@ -62,11 +48,4 @@
         </geometry>
       </collision>
-      <inertial>
-          <mass value="14.350897"/>
-          <origin xyz="-0.000007 0.221192 0.206856" rpy="0.0 0.0 0.0"/>
-          <inertia ixx="0.595207" ixy="0.000005" ixz="-0.000008"
-                                       iyy="0.625683" iyz="-0.003766"
-                                                           izz="0.059863"/>
-      </inertial>
     </link>
     <link name="${prefix}link_3">
@@ -74,5 +53,5 @@
         <origin xyz="0 0 0" rpy="0 0 0"/>
         <geometry>
-          <mesh filename="package://staubli_tx60_support/meshes/tx60/visual/link_3.stl"/>
+          <mesh filename="package://staubli_tx60_support/meshes/tx60l/visual/link_3.stl"/>
         </geometry>
         <xacro:material_staubli_ral_melon_yellow />
@@ -81,14 +60,7 @@
         <origin xyz="0 0 0" rpy="0 0 0"/>
         <geometry>
-          <mesh filename="package://staubli_tx60_support/meshes/tx60/collision/link_3.stl"/>
+          <mesh filename="package://staubli_tx60_support/meshes/tx60l/collision/link_3.stl"/>
         </geometry>
       </collision>
-      <inertial>
-          <mass value="7.501506"/>
-          <origin xyz="0.000002 0.065008 -0.071428" rpy="0.0 0.0 0.0"/>
-          <inertia ixx="0.058602" ixy="0.000000" ixz="0.000001"
-                                  iyy="0.056884" iyz="-0.003672"
-                                                 izz="0.034271"/>
-      </inertial>
     </link>
     <link name="${prefix}link_4">
@@ -106,11 +78,4 @@
         </geometry>
       </collision>
-      <inertial>
-          <mass value="6.420429"/>
-          <origin xyz="-0.001998 0.049992 0.360301" rpy="0.0 0.0 0.0"/>
-          <inertia ixx="0.103999" ixy="0.000003" ixz="-0.001379"
-                                  iyy="0.098782" iyz="-0.000007"
-                                                 izz="0.016071"/>
-      </inertial>
     </link>
     <link name="${prefix}link_5">
@@ -118,5 +83,5 @@
         <origin xyz="0 0 0" rpy="0 0 0"/>
         <geometry>
-          <mesh filename="package://staubli_tx60_support/meshes/tx60/visual/link_5.stl"/>
+          <mesh filename="package://staubli_tx60_support/meshes/tx60l/visual/link_5.stl"/>
         </geometry>
         <xacro:material_staubli_ral_grey_aluminium />
@@ -125,14 +90,7 @@
         <origin xyz="0 0 0" rpy="0 0 0"/>
         <geometry>
-          <mesh filename="package://staubli_tx60_support/meshes/tx60/collision/link_5.stl"/>
+          <mesh filename="package://staubli_tx60_support/meshes/tx60l/collision/link_5.stl"/>
         </geometry>
       </collision>
-      <inertial>
-          <mass value="0.568760"/>
-          <origin xyz="0.000000 0.049931 0.022823" rpy="0.0 0.0 0.0"/>
-          <inertia ixx="0.001084" ixy="0.000000" ixz="0.000000"
-                                  iyy="0.001123" iyz="0.000001"
-                                                 izz="0.000383"/>
-      </inertial>
     </link>
     <link name="${prefix}link_6">
@@ -140,5 +98,5 @@
         <origin xyz="0 0 0" rpy="0 0 0"/>
         <geometry>
-          <mesh filename="package://staubli_tx60_support/meshes/tx60/visual/link_6.stl"/>
+          <mesh filename="package://staubli_tx60_support/meshes/tx60l/visual/link_6.stl"/>
         </geometry>
         <xacro:material_staubli_ral_grey_aluminium />
@@ -147,17 +105,9 @@
         <origin xyz="0 0 0" rpy="0 0 0"/>
         <geometry>
-          <mesh filename="package://staubli_tx60_support/meshes/tx60/collision/link_6.stl"/>
+          <mesh filename="package://staubli_tx60_support/meshes/tx60l/collision/link_6.stl"/>
         </geometry>
       </collision>
-      <inertial>
-          <mass value="0.030977"/>
-          <origin xyz="-0.000243 0.050000 -0.206293" rpy="0.0 0.0 0.0"/>
-          <inertia ixx="0.000012" ixy="-0.000000" ixz="0.000000"
-                                  iyy="0.000011"  iyz="0.000000"
-                                                  izz="0.000022"/>
-      </inertial>
     </link>
-    <link name="${prefix}tool0"/>
-    <!-- joints -->
+    <!-- joints: main serial chain -->
     <joint name="${prefix}joint_1" type="revolute">
       <origin xyz="0 0 0.478" rpy="0 0 0"/>
@@ -168,5 +118,5 @@
       (1) effort limit = 318 Nm if floor mounted
       (2) effort limit = 111 Nm if wall mounted -->
-      <limit lower="-3.14159" upper="3.14159" effort="318.0" velocity="3.75" />
+      <limit lower="${radians(-180)}" upper="${radians(180)}" effort="0.0" velocity="${radians(435)}" />
       <dynamics damping="0.0" friction="0.0"/>
     </joint>
@@ -176,13 +126,13 @@
       <child link="${prefix}link_2"/>
       <axis xyz="0 1 0"/>
-      <limit lower="-2.268928" upper="2.574360" effort="130.0" velocity="2.97" />
+      <limit lower="${radians(-127.5)}" upper="${radians(127.5)}" effort="0.0" velocity="${radians(385)}" />
       <dynamics damping="0.0" friction="0.0"/>
     </joint>
     <joint name="${prefix}joint_3" type="revolute">
-      <origin xyz="0 0.05 0.500" rpy="0 0 0"/>
+      <origin xyz="0 0.05 0.425" rpy="0 0 0"/>
       <parent link="${prefix}link_2"/>
       <child link="${prefix}link_3"/>
       <axis xyz="0 1 0"/>
-      <limit lower="-2.530727" upper="2.530727" effort="65.0" velocity="4.45" />
+      <limit lower="${radians(-152.5)}" upper="${radians(152.5)}" effort="0.0" velocity="${radians(500)}" />
       <dynamics damping="0.0" friction="0.0"/>
     </joint>
@@ -192,13 +142,13 @@
       <child link="${prefix}link_4"/>
       <axis xyz="0 0 1"/>
-      <limit lower="-4.712389" upper="4.712389" effort="34.0" velocity="7.50" />
+      <limit lower="${radians(-270.0)}" upper="${radians(270.0)}" effort="0.0" velocity="${radians(995)}" />
       <dynamics damping="0.0" friction="0.0"/>
     </joint>
     <joint name="${prefix}joint_5" type="revolute">
-      <origin xyz="0 0 0.550" rpy="0 0 0"/>
+      <origin xyz="0 0 0.425" rpy="0 0 0"/>
       <parent link="${prefix}link_4"/>
       <child link="${prefix}link_5"/>
       <axis xyz="0 1 0"/>
-      <limit lower="-2.007129" upper="2.443461" effort="29.0" velocity="6.11" />
+      <limit lower="${radians(-122.5)}" upper="${radians(132.5)}" effort="0.0" velocity="${radians(1065)}" />
       <dynamics damping="0.0" friction="0.0"/>
     </joint>
@@ -208,11 +158,27 @@
       <child link="${prefix}link_6"/>
       <axis xyz="0 0 1"/>
-      <limit lower="-4.712389" upper="4.712389" effort="11.0" velocity="10.47" />
+      <limit lower="${radians(-270.0)}" upper="${radians(270.0)}" effort="0.0" velocity="${radians(1445)}" />
       <dynamics damping="0.0" friction="0.0"/>
     </joint>
-    <joint name="${prefix}joint_6-tool0" type="fixed">
-      <parent link="${prefix}link_6"/>
-      <child link="${prefix}tool0"/>
-      <origin xyz="0 0 0" rpy="0 0 0"/>
+    <!-- ROS-Industrial 'base' frame: base_link to Fanuc World Coordinates transform -->
+    <link name="${prefix}base" />
+    <joint name="${prefix}base_link-base" type="fixed">
+      <origin xyz="0 0 0.650" rpy="0 0 0"/>
+      <parent link="${prefix}base_link"/>
+      <child link="${prefix}base"/>
+    </joint>
+    <!-- ROS-Industrial 'flange' frame: attachment point for EEF models -->
+    <link name="${prefix}flange" />
+    <joint name="${prefix}joint_6-flange" type="fixed">
+      <origin xyz="0 0 0" rpy="0 0 0" />
+      <parent link="${prefix}link_6" />
+      <child link="${prefix}flange" />
+    </joint>
+    <!-- ROS-Industrial 'tool0' frame: all-zeros tool frame -->
+    <link name="${prefix}tool0" />
+    <joint name="${prefix}link_6-tool0" type="fixed">
+      <origin xyz="0 0 0" rpy="0 0 0" />
+      <parent link="${prefix}link_6" />
+      <child link="${prefix}tool0" />
     </joint>
   </xacro:macro>

Commit message: Added dimensions of tx60 to URDF file

File: staubli_tx60_support/urdf/tx60_macro.xacro (robot description, xacro)
@@ -111,5 +111,5 @@
     <!-- joints: main serial chain -->
     <joint name="${prefix}joint_1" type="revolute">
-      <origin xyz="0 0 0.478" rpy="0 0 0"/>
+      <origin xyz="0 0 0.375" rpy="0 0 0"/>
       <parent link="${prefix}base_link"/>
       <child link="${prefix}link_1"/>
@@ -122,5 +122,5 @@
     </joint>
     <joint name="${prefix}joint_2" type="revolute">
-      <origin xyz="0.050 0 0" rpy="0 0 0"/>
+      <origin xyz="0 0 0" rpy="0 0 0"/>
       <parent link="${prefix}link_1"/>
       <child link="${prefix}link_2"/>
@@ -130,5 +130,5 @@
     </joint>
     <joint name="${prefix}joint_3" type="revolute">
-      <origin xyz="0 0.05 0.425" rpy="0 0 0"/>
+      <origin xyz="0 0.02 0.290" rpy="0 0 0"/>
       <parent link="${prefix}link_2"/>
       <child link="${prefix}link_3"/>
@@ -146,5 +146,5 @@
     </joint>
     <joint name="${prefix}joint_5" type="revolute">
-      <origin xyz="0 0 0.425" rpy="0 0 0"/>
+      <origin xyz="0 0 0.310" rpy="0 0 0"/>
       <parent link="${prefix}link_4"/>
       <child link="${prefix}link_5"/>
@@ -154,5 +154,5 @@
     </joint>
     <joint name="${prefix}joint_6" type="revolute">
-      <origin xyz="0 0 0.100" rpy="0 0 0"/>
+      <origin xyz="0 0 0.07" rpy="0 0 0"/>
       <parent link="${prefix}link_5"/>
       <child link="${prefix}link_6"/>

Commit message: Updated the frames: base, flange and tool0 regarding the REP for industrial robots

File: staubli_tx60_support/urdf/tx60_macro.xacro (robot description, xacro)
@@ -164,5 +164,5 @@
     <link name="${prefix}base" />
     <joint name="${prefix}base_link-base" type="fixed">
-      <origin xyz="0 0 0.650" rpy="0 0 0"/>
+      <origin xyz="0 0 0" rpy="0 0 0"/>
       <parent link="${prefix}base_link"/>
       <child link="${prefix}base"/>
@@ -171,5 +171,5 @@
     <link name="${prefix}flange" />
     <joint name="${prefix}joint_6-flange" type="fixed">
-      <origin xyz="0 0 0" rpy="0 0 0" />
+      <origin xyz="0 0 0" rpy="0 ${radians(-90.0)} 0" />
       <parent link="${prefix}link_6" />
       <child link="${prefix}flange" />
@@ -177,7 +177,7 @@
     <!-- ROS-Industrial 'tool0' frame: all-zeros tool frame -->
     <link name="${prefix}tool0" />
-    <joint name="${prefix}link_6-tool0" type="fixed">
-      <origin xyz="0 0 0" rpy="0 0 0" />
-      <parent link="${prefix}link_6" />
+    <joint name="${prefix}flange-tool0" type="fixed">
+      <origin xyz="0 0 0" rpy="0 ${radians(90.0)} 0" />
+      <parent link="${prefix}flange" />
       <child link="${prefix}tool0" />
     </joint>

File: staubli_tx60_support/urdf/tx60l_macro.xacro (robot description, xacro)
@@ -164,5 +164,5 @@
     <link name="${prefix}base" />
     <joint name="${prefix}base_link-base" type="fixed">
-      <origin xyz="0 0 0.650" rpy="0 0 0"/>
+      <origin xyz="0 0 0" rpy="0 0 0"/>
       <parent link="${prefix}base_link"/>
       <child link="${prefix}base"/>
@@ -171,5 +171,5 @@
     <link name="${prefix}flange" />
     <joint name="${prefix}joint_6-flange" type="fixed">
-      <origin xyz="0 0 0" rpy="0 0 0" />
+      <origin xyz="0 0 0" rpy="0 ${radians(-90.0)} 0" />
       <parent link="${prefix}link_6" />
       <child link="${prefix}flange" />
@@ -177,7 +177,7 @@
     <!-- ROS-Industrial 'tool0' frame: all-zeros tool frame -->
     <link name="${prefix}tool0" />
-    <joint name="${prefix}link_6-tool0" type="fixed">
-      <origin xyz="0 0 0" rpy="0 0 0" />
-      <parent link="${prefix}link_6" />
+    <joint name="${prefix}flange-tool0" type="fixed">
+      <origin xyz="0 0 0" rpy="0 ${radians(90.0)} 0" />
+      <parent link="${prefix}flange" />
       <child link="${prefix}tool0" />
     </joint>

Commit message: Added gazebo simulation for tx60 series and added masses and inertia matrices for tx60 robot

File: staubli_tx60_support/urdf/tx60_macro.xacro (robot description, xacro)
@@ -18,4 +18,11 @@
         </geometry>
       </collision>
+      <inertial>
+          <mass value="4.65972258"/>
+          <origin xyz="-0.00257355 -0.00039402 0.08786146" rpy="0.0 0.0 0.0"/>
+          <inertia ixx="0.02319782" ixy="0.00023234" ixz="0.00162421"
+                                    iyy="0.02621324" iyz="0.00008092"
+                                                     izz="0.02286304"/>
+      </inertial>
     </link>
     <link name="${prefix}link_1">
@@ -33,4 +40,11 @@
         </geometry>
       </collision>
+<inertial>
+          <mass value="6.99103376"/>
+          <origin xyz="0.00000000 0.02467680 -0.05265925" rpy="0.0 0.0 0.0"/>
+          <inertia ixx="0.05672953" ixy="0.00000037" ixz="-0.00000049"
+                                    iyy="0.04909238" iyz="0.01016069"
+                                                     izz="0.03457565"/>
+      </inertial>
     </link>
     <link name="${prefix}link_2">
@@ -48,4 +62,11 @@
         </geometry>
       </collision>
+<inertial>
+          <mass value="4.29177000"/>
+          <origin xyz="-0.00000313 0.17159103 0.12393869" rpy="0.0 0.0 0.0"/>
+          <inertia ixx="0.07028551" ixy="0.00000037" ixz="-0.00000033"
+                                    iyy="0.07597923" iyz="-0.00033734"
+                                                     izz="0.00928775"/>
+      </inertial>
     </link>
     <link name="${prefix}link_3">
@@ -63,4 +84,11 @@
         </geometry>
       </collision>
+      <inertial>
+          <mass value="4.52768000"/>
+          <origin xyz="0.00424668 0.02553862 -0.00735408" rpy="0.0 0.0 0.0"/>
+          <inertia ixx="0.02469218" ixy="0.00032528" ixz="0.00063194"
+                                    iyy="0.02222651" iyz="-0.00155762"
+                                                     izz="0.01657366"/>
+      </inertial>
     </link>
     <link name="${prefix}link_4">
@@ -78,4 +106,11 @@
         </geometry>
       </collision>
+      <inertial>
+          <mass value="2.16976000"/>
+          <origin xyz="-0.00156932 0.00000000 0.21400361" rpy="0.0 0.0 0.0"/>
+          <inertia ixx="0.01161479" ixy="0.00000000" ixz="-0.00034929"
+                                    iyy="0.01033617" iyz="0.00000001"
+                                                     izz="0.00409557"/>
+      </inertial>
     </link>
     <link name="${prefix}link_5">
@@ -93,4 +128,11 @@
         </geometry>
       </collision>
+      <inertial>
+          <mass value="0.16254714"/>
+          <origin xyz="-0.00000105 0.00000000 0.01268974" rpy="0.0 0.0 0.0"/>
+          <inertia ixx="0.00012557" ixy="0.00000000" ixz="0.00000000"
+                                    iyy="0.00013289" iyz="0.00000000"
+                                                     izz="0.00006342"/>
+      </inertial>
     </link>
     <link name="${prefix}link_6">
@@ -108,4 +150,11 @@
         </geometry>
       </collision>
+      <inertial>
+          <mass value="0.00820000"/>
+          <origin xyz="-0.00022629 0.00000000 -0.00597808" rpy="0.0 0.0 0.0"/>
+          <inertia ixx="0.00000096" ixy="0.00000000" ixz="0.00000000"
+                                    iyy="0.00000093" iyz="0.00000000"
+                                                     izz="0.00000154"/>
+      </inertial>
     </link>
     <!-- joints: main serial chain -->
