Commit message: update xacros

File: staubli_tx260_support/urdf/tx260.xacro (robot description, xacro)
@@ -2,4 +2,4 @@
 <robot name="staubli_tx260" xmlns:xacro="http://wiki.ros.org/xacro">
   <xacro:include filename="$(find staubli_tx260_support)/urdf/tx260_macro.xacro"/>
-  <xacro:staubli_tx260l prefix=""/>
+  <xacro:staubli_tx260 prefix=""/>
 </robot>

File: staubli_tx260_support/urdf/tx260_macro.xacro (robot description, xacro)
@@ -179,5 +179,5 @@
     </joint>
     <joint name="${prefix}joint_3" type="revolute">
-      <origin xyz="0 0.02 0.40" rpy="0 0 0"/>
+      <origin xyz="0 0.02 0.29" rpy="0 0 0"/>
       <parent link="${prefix}link_2"/>
       <child link="${prefix}link_3"/>
@@ -195,5 +195,5 @@
     </joint>
     <joint name="${prefix}joint_5" type="revolute">
-      <origin xyz="0 0 0.45" rpy="0 0 0"/>
+      <origin xyz="0 0 0.31" rpy="0 0 0"/>
       <parent link="${prefix}link_4"/>
       <child link="${prefix}link_5"/>
