Commit message: renamed to follow REP-3, added missing files

File: staubli_tx2_90_support/urdf/tx2_90_macro.xacro (robot description, xacro)
@@ -2,5 +2,5 @@
 <robot xmlns:xacro="http://wiki.ros.org/xacro">
   <xacro:include filename="$(find staubli_resources)/urdf/common_materials.xacro"/>
-  <xacro:macro name="staubli_tx2-90xl" params="prefix">
+  <xacro:macro name="staubli_tx2_90" params="prefix">
     <!-- links: main serial chain -->
     <link name="${prefix}base_link">
@@ -8,12 +8,12 @@
         <origin xyz="0 0 0" rpy="0 0 0"/>
         <geometry>
-          <mesh filename="package://staubli_tx2-90_support/meshes/tx2-90/visual/base_link.stl"/>
-        </geometry>
-        <xacro:material_staubli_ral_melon_yellow />
-      </visual>
-      <collision>
-        <origin xyz="0 0 0" rpy="0 0 0"/>
-        <geometry>
-          <mesh filename="package://staubli_tx2-90_support/meshes/tx2-90/collision/base_link.stl"/>
+          <mesh filename="package://staubli_tx2_90_support/meshes/tx2_90/visual/base_link.stl"/>
+        </geometry>
+        <xacro:material_staubli_ral_melon_yellow />
+      </visual>
+      <collision>
+        <origin xyz="0 0 0" rpy="0 0 0"/>
+        <geometry>
+          <mesh filename="package://staubli_tx2_90_support/meshes/tx2_90/collision/base_link.stl"/>
         </geometry>
       </collision>
@@ -30,12 +30,12 @@
         <origin xyz="0 0 0" rpy="0 0 0"/>
         <geometry>
-          <mesh filename="package://staubli_tx2-90_support/meshes/tx2-90/visual/link_1.stl"/>
-        </geometry>
-        <xacro:material_staubli_ral_melon_yellow />
-      </visual>
-      <collision>
-        <origin xyz="0 0 0" rpy="0 0 0"/>
-        <geometry>
-          <mesh filename="package://staubli_tx2-90_support/meshes/tx2-90/collision/link_1.stl"/>
+          <mesh filename="package://staubli_tx2_90_support/meshes/tx2_90/visual/link_1.stl"/>
+        </geometry>
+        <xacro:material_staubli_ral_melon_yellow />
+      </visual>
+      <collision>
+        <origin xyz="0 0 0" rpy="0 0 0"/>
+        <geometry>
+          <mesh filename="package://staubli_tx2_90_support/meshes/tx2_90/collision/link_1.stl"/>
         </geometry>
       </collision>
@@ -52,12 +52,12 @@
         <origin xyz="0 0 0" rpy="0 0 0"/>
         <geometry>
-          <mesh filename="package://staubli_tx2-90_support/meshes/tx2-90xl/visual/link_2.stl"/>
-        </geometry>
-        <xacro:material_staubli_ral_melon_yellow />
-      </visual>
-      <collision>
-        <origin xyz="0 0 0" rpy="0 0 0"/>
-        <geometry>
-          <mesh filename="package://staubli_tx2-90_support/meshes/tx2-90xl/collision/link_2.stl"/>
+          <mesh filename="package://staubli_tx2_90_support/meshes/tx2_90/visual/link_2.stl"/>
+        </geometry>
+        <xacro:material_staubli_ral_melon_yellow />
+      </visual>
+      <collision>
+        <origin xyz="0 0 0" rpy="0 0 0"/>
+        <geometry>
+          <mesh filename="package://staubli_tx2_90_support/meshes/tx2_90/collision/link_2.stl"/>
         </geometry>
       </collision>
@@ -74,12 +74,12 @@
         <origin xyz="0 0 0" rpy="0 0 0"/>
         <geometry>
-          <mesh filename="package://staubli_tx2-90_support/meshes/tx2-90/visual/link_3.stl"/>
-        </geometry>
-        <xacro:material_staubli_ral_melon_yellow />
-      </visual>
-      <collision>
-        <origin xyz="0 0 0" rpy="0 0 0"/>
-        <geometry>
-          <mesh filename="package://staubli_tx2-90_support/meshes/tx2-90/collision/link_3.stl"/>
+          <mesh filename="package://staubli_tx2_90_support/meshes/tx2_90/visual/link_3.stl"/>
+        </geometry>
+        <xacro:material_staubli_ral_melon_yellow />
+      </visual>
+      <collision>
+        <origin xyz="0 0 0" rpy="0 0 0"/>
+        <geometry>
+          <mesh filename="package://staubli_tx2_90_support/meshes/tx2_90/collision/link_3.stl"/>
         </geometry>
       </collision>
@@ -96,12 +96,12 @@
         <origin xyz="0 0 0" rpy="0 0 0"/>
         <geometry>
-          <mesh filename="package://staubli_tx2-90_support/meshes/tx2-90xl/visual/link_4.stl"/>
-        </geometry>
-        <xacro:material_staubli_ral_melon_yellow />
-      </visual>
-      <collision>
-        <origin xyz="0 0 0" rpy="0 0 0"/>
-        <geometry>
-          <mesh filename="package://staubli_tx2-90_support/meshes/tx2-90xl/collision/link_4.stl"/>
+          <mesh filename="package://staubli_tx2_90_support/meshes/tx2_90/visual/link_4.stl"/>
+        </geometry>
+        <xacro:material_staubli_ral_melon_yellow />
+      </visual>
+      <collision>
+        <origin xyz="0 0 0" rpy="0 0 0"/>
+        <geometry>
+          <mesh filename="package://staubli_tx2_90_support/meshes/tx2_90/collision/link_4.stl"/>
         </geometry>
       </collision>
@@ -118,5 +118,5 @@
         <origin xyz="0 0 0" rpy="0 0 0"/>
         <geometry>
-          <mesh filename="package://staubli_tx2-90_support/meshes/tx2-90/visual/link_5.stl"/>
+          <mesh filename="package://staubli_tx2_90_support/meshes/tx2_90/visual/link_5.stl"/>
         </geometry>
         <xacro:material_staubli_ral_grey_aluminium />
@@ -125,5 +125,5 @@
         <origin xyz="0 0 0" rpy="0 0 0"/>
         <geometry>
-          <mesh filename="package://staubli_tx2-90_support/meshes/tx2-90/collision/link_5.stl"/>
+          <mesh filename="package://staubli_tx2_90_support/meshes/tx2_90/collision/link_5.stl"/>
         </geometry>
       </collision>
@@ -140,5 +140,5 @@
         <origin xyz="0 0 0" rpy="0 0 0"/>
         <geometry>
-          <mesh filename="package://staubli_tx2-90_support/meshes/tx2-90/visual/link_6.stl"/>
+          <mesh filename="package://staubli_tx2_90_support/meshes/tx2_90/visual/link_6.stl"/>
         </geometry>
         <xacro:material_staubli_ral_grey_aluminium />
@@ -147,5 +147,5 @@
         <origin xyz="0 0 0" rpy="0 0 0"/>
         <geometry>
-          <mesh filename="package://staubli_tx2-90_support/meshes/tx2-90/collision/link_6.stl"/>
+          <mesh filename="package://staubli_tx2_90_support/meshes/tx2_90/collision/link_6.stl"/>
         </geometry>
       </collision>
@@ -179,5 +179,5 @@
     </joint>
     <joint name="${prefix}joint_3" type="revolute">
-      <origin xyz="0 0.05 0.650" rpy="0 0 0"/>
+      <origin xyz="0 0.05 0.425" rpy="0 0 0"/>
       <parent link="${prefix}link_2"/>
       <child link="${prefix}link_3"/>
@@ -195,5 +195,5 @@
     </joint>
     <joint name="${prefix}joint_5" type="revolute">
-      <origin xyz="0 0 0.650" rpy="0 0 0"/>
+      <origin xyz="0 0 0.425" rpy="0 0 0"/>
       <parent link="${prefix}link_4"/>
       <child link="${prefix}link_5"/>

File: staubli_tx2_90_support/urdf/tx2_90l_macro.xacro (robot description, xacro)
@@ -2,5 +2,5 @@
 <robot xmlns:xacro="http://wiki.ros.org/xacro">
   <xacro:include filename="$(find staubli_resources)/urdf/common_materials.xacro"/>
-  <xacro:macro name="staubli_tx2-90" params="prefix">
+  <xacro:macro name="staubli_tx2_90l" params="prefix">
     <!-- links: main serial chain -->
     <link name="${prefix}base_link">
@@ -8,12 +8,12 @@
         <origin xyz="0 0 0" rpy="0 0 0"/>
         <geometry>
-          <mesh filename="package://staubli_tx2-90_support/meshes/tx2-90/visual/base_link.stl"/>
-        </geometry>
-        <xacro:material_staubli_ral_melon_yellow />
-      </visual>
-      <collision>
-        <origin xyz="0 0 0" rpy="0 0 0"/>
-        <geometry>
-          <mesh filename="package://staubli_tx2-90_support/meshes/tx2-90/collision/base_link.stl"/>
+          <mesh filename="package://staubli_tx2_90_support/meshes/tx2_90/visual/base_link.stl"/>
+        </geometry>
+        <xacro:material_staubli_ral_melon_yellow />
+      </visual>
+      <collision>
+        <origin xyz="0 0 0" rpy="0 0 0"/>
+        <geometry>
+          <mesh filename="package://staubli_tx2_90_support/meshes/tx2_90/collision/base_link.stl"/>
         </geometry>
       </collision>
@@ -30,12 +30,12 @@
         <origin xyz="0 0 0" rpy="0 0 0"/>
         <geometry>
-          <mesh filename="package://staubli_tx2-90_support/meshes/tx2-90/visual/link_1.stl"/>
-        </geometry>
-        <xacro:material_staubli_ral_melon_yellow />
-      </visual>
-      <collision>
-        <origin xyz="0 0 0" rpy="0 0 0"/>
-        <geometry>
-          <mesh filename="package://staubli_tx2-90_support/meshes/tx2-90/collision/link_1.stl"/>
+          <mesh filename="package://staubli_tx2_90_support/meshes/tx2_90/visual/link_1.stl"/>
+        </geometry>
+        <xacro:material_staubli_ral_melon_yellow />
+      </visual>
+      <collision>
+        <origin xyz="0 0 0" rpy="0 0 0"/>
+        <geometry>
+          <mesh filename="package://staubli_tx2_90_support/meshes/tx2_90/collision/link_1.stl"/>
         </geometry>
       </collision>
@@ -52,12 +52,12 @@
         <origin xyz="0 0 0" rpy="0 0 0"/>
         <geometry>
-          <mesh filename="package://staubli_tx2-90_support/meshes/tx2-90/visual/link_2.stl"/>
-        </geometry>
-        <xacro:material_staubli_ral_melon_yellow />
-      </visual>
-      <collision>
-        <origin xyz="0 0 0" rpy="0 0 0"/>
-        <geometry>
-          <mesh filename="package://staubli_tx2-90_support/meshes/tx2-90/collision/link_2.stl"/>
+          <mesh filename="package://staubli_tx2_90_support/meshes/tx2_90l/visual/link_2.stl"/>
+        </geometry>
+        <xacro:material_staubli_ral_melon_yellow />
+      </visual>
+      <collision>
+        <origin xyz="0 0 0" rpy="0 0 0"/>
+        <geometry>
+          <mesh filename="package://staubli_tx2_90_support/meshes/tx2_90l/collision/link_2.stl"/>
         </geometry>
       </collision>
@@ -74,12 +74,12 @@
         <origin xyz="0 0 0" rpy="0 0 0"/>
         <geometry>
-          <mesh filename="package://staubli_tx2-90_support/meshes/tx2-90/visual/link_3.stl"/>
-        </geometry>
-        <xacro:material_staubli_ral_melon_yellow />
-      </visual>
-      <collision>
-        <origin xyz="0 0 0" rpy="0 0 0"/>
-        <geometry>
-          <mesh filename="package://staubli_tx2-90_support/meshes/tx2-90/collision/link_3.stl"/>
+          <mesh filename="package://staubli_tx2_90_support/meshes/tx2_90/visual/link_3.stl"/>
+        </geometry>
+        <xacro:material_staubli_ral_melon_yellow />
+      </visual>
+      <collision>
+        <origin xyz="0 0 0" rpy="0 0 0"/>
+        <geometry>
+          <mesh filename="package://staubli_tx2_90_support/meshes/tx2_90/collision/link_3.stl"/>
         </geometry>
       </collision>
@@ -96,12 +96,12 @@
         <origin xyz="0 0 0" rpy="0 0 0"/>
         <geometry>
-          <mesh filename="package://staubli_tx2-90_support/meshes/tx2-90/visual/link_4.stl"/>
-        </geometry>
-        <xacro:material_staubli_ral_melon_yellow />
-      </visual>
-      <collision>
-        <origin xyz="0 0 0" rpy="0 0 0"/>
-        <geometry>
-          <mesh filename="package://staubli_tx2-90_support/meshes/tx2-90/collision/link_4.stl"/>
+          <mesh filename="package://staubli_tx2_90_support/meshes/tx2_90l/visual/link_4.stl"/>
+        </geometry>
+        <xacro:material_staubli_ral_melon_yellow />
+      </visual>
+      <collision>
+        <origin xyz="0 0 0" rpy="0 0 0"/>
+        <geometry>
+          <mesh filename="package://staubli_tx2_90_support/meshes/tx2_90l/collision/link_4.stl"/>
         </geometry>
       </collision>
@@ -118,5 +118,5 @@
         <origin xyz="0 0 0" rpy="0 0 0"/>
         <geometry>
-          <mesh filename="package://staubli_tx2-90_support/meshes/tx2-90/visual/link_5.stl"/>
+          <mesh filename="package://staubli_tx2_90_support/meshes/tx2_90/visual/link_5.stl"/>
         </geometry>
         <xacro:material_staubli_ral_grey_aluminium />
@@ -125,5 +125,5 @@
         <origin xyz="0 0 0" rpy="0 0 0"/>
         <geometry>
-          <mesh filename="package://staubli_tx2-90_support/meshes/tx2-90/collision/link_5.stl"/>
+          <mesh filename="package://staubli_tx2_90_support/meshes/tx2_90/collision/link_5.stl"/>
         </geometry>
       </collision>
@@ -140,5 +140,5 @@
         <origin xyz="0 0 0" rpy="0 0 0"/>
         <geometry>
-          <mesh filename="package://staubli_tx2-90_support/meshes/tx2-90/visual/link_6.stl"/>
+          <mesh filename="package://staubli_tx2_90_support/meshes/tx2_90/visual/link_6.stl"/>
         </geometry>
         <xacro:material_staubli_ral_grey_aluminium />
@@ -147,5 +147,5 @@
         <origin xyz="0 0 0" rpy="0 0 0"/>
         <geometry>
-          <mesh filename="package://staubli_tx2-90_support/meshes/tx2-90/collision/link_6.stl"/>
+          <mesh filename="package://staubli_tx2_90_support/meshes/tx2_90/collision/link_6.stl"/>
         </geometry>
       </collision>
@@ -179,5 +179,5 @@
     </joint>
     <joint name="${prefix}joint_3" type="revolute">
-      <origin xyz="0 0.05 0.425" rpy="0 0 0"/>
+      <origin xyz="0 0.05 0.500" rpy="0 0 0"/>
       <parent link="${prefix}link_2"/>
       <child link="${prefix}link_3"/>
@@ -195,5 +195,5 @@
     </joint>
     <joint name="${prefix}joint_5" type="revolute">
-      <origin xyz="0 0 0.425" rpy="0 0 0"/>
+      <origin xyz="0 0 0.550" rpy="0 0 0"/>
       <parent link="${prefix}link_4"/>
       <child link="${prefix}link_5"/>

File: staubli_tx2_90_support/urdf/tx2_90xl_macro.xacro (robot description, xacro)
@@ -2,5 +2,5 @@
 <robot xmlns:xacro="http://wiki.ros.org/xacro">
   <xacro:include filename="$(find staubli_resources)/urdf/common_materials.xacro"/>
-  <xacro:macro name="staubli_tx2-90l" params="prefix">
+  <xacro:macro name="staubli_tx2_90xl" params="prefix">
     <!-- links: main serial chain -->
     <link name="${prefix}base_link">
@@ -8,12 +8,12 @@
         <origin xyz="0 0 0" rpy="0 0 0"/>
         <geometry>
-          <mesh filename="package://staubli_tx2-90_support/meshes/tx2-90/visual/base_link.stl"/>
-        </geometry>
-        <xacro:material_staubli_ral_melon_yellow />
-      </visual>
-      <collision>
-        <origin xyz="0 0 0" rpy="0 0 0"/>
-        <geometry>
-          <mesh filename="package://staubli_tx2-90_support/meshes/tx2-90/collision/base_link.stl"/>
+          <mesh filename="package://staubli_tx2_90_support/meshes/tx2_90/visual/base_link.stl"/>
+        </geometry>
+        <xacro:material_staubli_ral_melon_yellow />
+      </visual>
+      <collision>
+        <origin xyz="0 0 0" rpy="0 0 0"/>
+        <geometry>
+          <mesh filename="package://staubli_tx2_90_support/meshes/tx2_90/collision/base_link.stl"/>
         </geometry>
       </collision>
@@ -30,12 +30,12 @@
         <origin xyz="0 0 0" rpy="0 0 0"/>
         <geometry>
-          <mesh filename="package://staubli_tx2-90_support/meshes/tx2-90/visual/link_1.stl"/>
-        </geometry>
-        <xacro:material_staubli_ral_melon_yellow />
-      </visual>
-      <collision>
-        <origin xyz="0 0 0" rpy="0 0 0"/>
-        <geometry>
-          <mesh filename="package://staubli_tx2-90_support/meshes/tx2-90/collision/link_1.stl"/>
+          <mesh filename="package://staubli_tx2_90_support/meshes/tx2_90/visual/link_1.stl"/>
+        </geometry>
+        <xacro:material_staubli_ral_melon_yellow />
+      </visual>
+      <collision>
+        <origin xyz="0 0 0" rpy="0 0 0"/>
+        <geometry>
+          <mesh filename="package://staubli_tx2_90_support/meshes/tx2_90/collision/link_1.stl"/>
         </geometry>
       </collision>
@@ -52,12 +52,12 @@
         <origin xyz="0 0 0" rpy="0 0 0"/>
         <geometry>
-          <mesh filename="package://staubli_tx2-90_support/meshes/tx2-90l/visual/link_2.stl"/>
-        </geometry>
-        <xacro:material_staubli_ral_melon_yellow />
-      </visual>
-      <collision>
-        <origin xyz="0 0 0" rpy="0 0 0"/>
-        <geometry>
-          <mesh filename="package://staubli_tx2-90_support/meshes/tx2-90l/collision/link_2.stl"/>
+          <mesh filename="package://staubli_tx2_90_support/meshes/tx2_90xl/visual/link_2.stl"/>
+        </geometry>
+        <xacro:material_staubli_ral_melon_yellow />
+      </visual>
+      <collision>
+        <origin xyz="0 0 0" rpy="0 0 0"/>
+        <geometry>
+          <mesh filename="package://staubli_tx2_90_support/meshes/tx2_90xl/collision/link_2.stl"/>
         </geometry>
       </collision>
@@ -74,12 +74,12 @@
         <origin xyz="0 0 0" rpy="0 0 0"/>
         <geometry>
-          <mesh filename="package://staubli_tx2-90_support/meshes/tx2-90/visual/link_3.stl"/>
-        </geometry>
-        <xacro:material_staubli_ral_melon_yellow />
-      </visual>
-      <collision>
-        <origin xyz="0 0 0" rpy="0 0 0"/>
-        <geometry>
-          <mesh filename="package://staubli_tx2-90_support/meshes/tx2-90/collision/link_3.stl"/>
+          <mesh filename="package://staubli_tx2_90_support/meshes/tx2_90/visual/link_3.stl"/>
+        </geometry>
+        <xacro:material_staubli_ral_melon_yellow />
+      </visual>
+      <collision>
+        <origin xyz="0 0 0" rpy="0 0 0"/>
+        <geometry>
+          <mesh filename="package://staubli_tx2_90_support/meshes/tx2_90/collision/link_3.stl"/>
         </geometry>
       </collision>
@@ -96,12 +96,12 @@
         <origin xyz="0 0 0" rpy="0 0 0"/>
         <geometry>
-          <mesh filename="package://staubli_tx2-90_support/meshes/tx2-90l/visual/link_4.stl"/>
-        </geometry>
-        <xacro:material_staubli_ral_melon_yellow />
-      </visual>
-      <collision>
-        <origin xyz="0 0 0" rpy="0 0 0"/>
-        <geometry>
-          <mesh filename="package://staubli_tx2-90_support/meshes/tx2-90l/collision/link_4.stl"/>
+          <mesh filename="package://staubli_tx2_90_support/meshes/tx2_90xl/visual/link_4.stl"/>
+        </geometry>
+        <xacro:material_staubli_ral_melon_yellow />
+      </visual>
+      <collision>
+        <origin xyz="0 0 0" rpy="0 0 0"/>
+        <geometry>
+          <mesh filename="package://staubli_tx2_90_support/meshes/tx2_90xl/collision/link_4.stl"/>
         </geometry>
       </collision>
@@ -118,5 +118,5 @@
         <origin xyz="0 0 0" rpy="0 0 0"/>
         <geometry>
-          <mesh filename="package://staubli_tx2-90_support/meshes/tx2-90/visual/link_5.stl"/>
+          <mesh filename="package://staubli_tx2_90_support/meshes/tx2_90/visual/link_5.stl"/>
         </geometry>
         <xacro:material_staubli_ral_grey_aluminium />
@@ -125,5 +125,5 @@
         <origin xyz="0 0 0" rpy="0 0 0"/>
         <geometry>
-          <mesh filename="package://staubli_tx2-90_support/meshes/tx2-90/collision/link_5.stl"/>
+          <mesh filename="package://staubli_tx2_90_support/meshes/tx2_90/collision/link_5.stl"/>
         </geometry>
       </collision>
@@ -140,5 +140,5 @@
         <origin xyz="0 0 0" rpy="0 0 0"/>
         <geometry>
-          <mesh filename="package://staubli_tx2-90_support/meshes/tx2-90/visual/link_6.stl"/>
+          <mesh filename="package://staubli_tx2_90_support/meshes/tx2_90/visual/link_6.stl"/>
         </geometry>
         <xacro:material_staubli_ral_grey_aluminium />
@@ -147,5 +147,5 @@
         <origin xyz="0 0 0" rpy="0 0 0"/>
         <geometry>
-          <mesh filename="package://staubli_tx2-90_support/meshes/tx2-90/collision/link_6.stl"/>
+          <mesh filename="package://staubli_tx2_90_support/meshes/tx2_90/collision/link_6.stl"/>
         </geometry>
       </collision>
@@ -179,5 +179,5 @@
     </joint>
     <joint name="${prefix}joint_3" type="revolute">
-      <origin xyz="0 0.05 0.500" rpy="0 0 0"/>
+      <origin xyz="0 0.05 0.650" rpy="0 0 0"/>
       <parent link="${prefix}link_2"/>
       <child link="${prefix}link_3"/>
@@ -195,5 +195,5 @@
     </joint>
     <joint name="${prefix}joint_5" type="revolute">
-      <origin xyz="0 0 0.550" rpy="0 0 0"/>
+      <origin xyz="0 0 0.650" rpy="0 0 0"/>
       <parent link="${prefix}link_4"/>
       <child link="${prefix}link_5"/>
