Commit message: Formatting and reordering xacro

File: staubli_tx2_90_support/urdf/tx2_90_macro.xacro (robot description, xacro)
@@ -66,6 +66,6 @@
           <origin xyz="-0.000007 0.221192 0.206856" rpy="0.0 0.0 0.0"/>
           <inertia ixx="0.595207" ixy="0.000005" ixz="-0.000008"
-                                       iyy="0.625683" iyz="-0.003766"
-                                                           izz="0.059863"/>
+                                  iyy="0.625683" iyz="-0.003766"
+                                                 izz="0.059863"/>
       </inertial>
     </link>
@@ -210,9 +210,4 @@
       <dynamics damping="0.0" friction="0.0"/>
     </joint>
-    <joint name="${prefix}joint_6-tool0" type="fixed">
-      <parent link="${prefix}link_6"/>
-      <child link="${prefix}tool0"/>
-      <origin xyz="0 0 0" rpy="0 0 0"/>
-    </joint>
     <!-- ROS-Industrial 'base' frame: base_link to Staubli World Coordinates transform -->
     <link name="${prefix}base" />
@@ -231,4 +226,9 @@
     <!-- ROS-Industrial 'tool0' frame: all-zeros tool frame -->
     <link name="${prefix}tool0" />
+    <joint name="${prefix}joint_6-tool0" type="fixed">
+      <parent link="${prefix}link_6"/>
+      <child link="${prefix}tool0"/>
+      <origin xyz="0 0 0" rpy="0 0 0"/>
+    </joint>
   </xacro:macro>
 </robot>

File: staubli_tx2_90_support/urdf/tx2_90l_macro.xacro (robot description, xacro)
@@ -66,6 +66,6 @@
           <origin xyz="-0.000007 0.221192 0.206856" rpy="0.0 0.0 0.0"/>
           <inertia ixx="0.595207" ixy="0.000005" ixz="-0.000008"
-                                       iyy="0.625683" iyz="-0.003766"
-                                                           izz="0.059863"/>
+                                  iyy="0.625683" iyz="-0.003766"
+                                                 izz="0.059863"/>
       </inertial>
     </link>
@@ -210,9 +210,4 @@
       <dynamics damping="0.0" friction="0.0"/>
     </joint>
-    <joint name="${prefix}joint_6-tool0" type="fixed">
-      <parent link="${prefix}link_6"/>
-      <child link="${prefix}tool0"/>
-      <origin xyz="0 0 0" rpy="0 0 0"/>
-    </joint>
     <!-- ROS-Industrial 'base' frame: base_link to Staubli World Coordinates transform -->
     <link name="${prefix}base" />
@@ -231,4 +226,9 @@
     <!-- ROS-Industrial 'tool0' frame: all-zeros tool frame -->
     <link name="${prefix}tool0" />
+        <joint name="${prefix}joint_6-tool0" type="fixed">
+      <parent link="${prefix}link_6"/>
+      <child link="${prefix}tool0"/>
+      <origin xyz="0 0 0" rpy="0 0 0"/>
+    </joint>
   </xacro:macro>
 </robot>

File: staubli_tx2_90_support/urdf/tx2_90xl_macro.xacro (robot description, xacro)
@@ -66,6 +66,6 @@
           <origin xyz="-0.000007 0.221192 0.206856" rpy="0.0 0.0 0.0"/>
           <inertia ixx="0.595207" ixy="0.000005" ixz="-0.000008"
-                                       iyy="0.625683" iyz="-0.003766"
-                                                           izz="0.059863"/>
+                                  iyy="0.625683" iyz="-0.003766"
+                                                 izz="0.059863"/>
       </inertial>
     </link>
@@ -210,9 +210,4 @@
       <dynamics damping="0.0" friction="0.0"/>
     </joint>
-    <joint name="${prefix}joint_6-tool0" type="fixed">
-      <parent link="${prefix}link_6"/>
-      <child link="${prefix}tool0"/>
-      <origin xyz="0 0 0" rpy="0 0 0"/>
-    </joint>
     <!-- ROS-Industrial 'base' frame: base_link to Staubli World Coordinates transform -->
     <link name="${prefix}base" />
@@ -231,4 +226,9 @@
     <!-- ROS-Industrial 'tool0' frame: all-zeros tool frame -->
     <link name="${prefix}tool0" />
+    <joint name="${prefix}joint_6-tool0" type="fixed">
+      <parent link="${prefix}link_6"/>
+      <child link="${prefix}tool0"/>
+      <origin xyz="0 0 0" rpy="0 0 0"/>
+    </joint>
   </xacro:macro>
 </robot>

Commit message: remove copied inertial values

File: staubli_tx2_90_support/urdf/tx2_90_macro.xacro (robot description, xacro)
@@ -18,11 +18,4 @@
         </geometry>
       </collision>
-      <inertial>
-          <mass value="10.733459"/>
-          <origin xyz="0.014288 0.000001 0.122264" rpy="0.0 0.0 0.0"/>
-          <inertia ixx="0.096590" ixy="-0.000005" ixz="-0.003803"
-                                  iyy="0.087591"  iyz="-0.000001"
-                                                  izz="0.081632"/>
-      </inertial>
     </link>
     <link name="${prefix}link_1">
@@ -40,11 +33,4 @@
         </geometry>
       </collision>
-      <inertial>
-          <mass value="16.934564"/>
-          <origin xyz="0.019143 0.024764 -0.064596" rpy="0.0 0.0 0.0"/>
-          <inertia ixx="0.222318" ixy="0.016499" ixz="0.023794"
-                                  iyy="0.208959" iyz="0.031663"
-                                                 izz="0.157081"/>
-      </inertial>
     </link>
     <link name="${prefix}link_2">
@@ -62,11 +48,4 @@
         </geometry>
       </collision>
-      <inertial>
-          <mass value="14.350897"/>
-          <origin xyz="-0.000007 0.221192 0.206856" rpy="0.0 0.0 0.0"/>
-          <inertia ixx="0.595207" ixy="0.000005" ixz="-0.000008"
-                                  iyy="0.625683" iyz="-0.003766"
-                                                 izz="0.059863"/>
-      </inertial>
     </link>
     <link name="${prefix}link_3">
@@ -84,11 +63,4 @@
         </geometry>
       </collision>
-      <inertial>
-          <mass value="7.501506"/>
-          <origin xyz="0.000002 0.065008 -0.071428" rpy="0.0 0.0 0.0"/>
-          <inertia ixx="0.058902" ixy="0.000000" ixz="0.000001"
-                                  iyy="0.056884" iyz="-0.003672"
-                                                 izz="0.034271"/>
-      </inertial>
     </link>
     <link name="${prefix}link_4">
@@ -106,11 +78,4 @@
         </geometry>
       </collision>
-      <inertial>
-          <mass value="6.420429"/>
-          <origin xyz="-0.001998 0.049992 0.360301" rpy="0.0 0.0 0.0"/>
-          <inertia ixx="0.103999" ixy="0.000003" ixz="-0.001379"
-                                  iyy="0.098782" iyz="-0.000007"
-                                                 izz="0.019071"/>
-      </inertial>
     </link>
     <link name="${prefix}link_5">
@@ -128,11 +93,4 @@
         </geometry>
       </collision>
-      <inertial>
-          <mass value="0.568760"/>
-          <origin xyz="0.000000 0.049931 0.022823" rpy="0.0 0.0 0.0"/>
-          <inertia ixx="0.001084" ixy="0.000000" ixz="0.000000"
-                                  iyy="0.001123" iyz="0.000001"
-                                                 izz="0.000383"/>
-      </inertial>
     </link>
     <link name="${prefix}link_6">
@@ -150,11 +108,4 @@
         </geometry>
       </collision>
-      <inertial>
-          <mass value="0.030977"/>
-          <origin xyz="-0.000243 0.050000 -0.206293" rpy="0.0 0.0 0.0"/>
-          <inertia ixx="0.000012" ixy="-0.000000" ixz="0.000000"
-                                  iyy="0.000011"  iyz="0.000000"
-                                                  izz="0.000022"/>
-      </inertial>
     </link>
     <!-- joints: main serial chain -->

File: staubli_tx2_90_support/urdf/tx2_90l_macro.xacro (robot description, xacro)
@@ -18,11 +18,4 @@
         </geometry>
       </collision>
-      <inertial>
-          <mass value="10.733459"/>
-          <origin xyz="0.014288 0.000001 0.122264" rpy="0.0 0.0 0.0"/>
-          <inertia ixx="0.096590" ixy="-0.000005" ixz="-0.003803"
-                                  iyy="0.087591"  iyz="-0.000001"
-                                                  izz="0.081632"/>
-      </inertial>
     </link>
     <link name="${prefix}link_1">
@@ -40,11 +33,4 @@
         </geometry>
       </collision>
-      <inertial>
-          <mass value="16.934564"/>
-          <origin xyz="0.019143 0.024764 -0.064596" rpy="0.0 0.0 0.0"/>
-          <inertia ixx="0.222318" ixy="0.016499" ixz="0.023794"
-                                  iyy="0.208959" iyz="0.031663"
-                                                 izz="0.157081"/>
-      </inertial>
     </link>
     <link name="${prefix}link_2">
@@ -62,11 +48,4 @@
         </geometry>
       </collision>
-      <inertial>
-          <mass value="14.350897"/>
-          <origin xyz="-0.000007 0.221192 0.206856" rpy="0.0 0.0 0.0"/>
-          <inertia ixx="0.595207" ixy="0.000005" ixz="-0.000008"
-                                  iyy="0.625683" iyz="-0.003766"
-                                                 izz="0.059863"/>
-      </inertial>
     </link>
     <link name="${prefix}link_3">
@@ -84,11 +63,4 @@
         </geometry>
       </collision>
-      <inertial>
-          <mass value="7.501506"/>
-          <origin xyz="0.000002 0.065008 -0.071428" rpy="0.0 0.0 0.0"/>
-          <inertia ixx="0.058902" ixy="0.000000" ixz="0.000001"
-                                  iyy="0.056884" iyz="-0.003672"
-                                                 izz="0.034271"/>
-      </inertial>
     </link>
     <link name="${prefix}link_4">
@@ -106,11 +78,4 @@
         </geometry>
       </collision>
-      <inertial>
-          <mass value="6.420429"/>
-          <origin xyz="-0.001998 0.049992 0.360301" rpy="0.0 0.0 0.0"/>
-          <inertia ixx="0.103999" ixy="0.000003" ixz="-0.001379"
-                                  iyy="0.098782" iyz="-0.000007"
-                                                 izz="0.019071"/>
-      </inertial>
     </link>
     <link name="${prefix}link_5">
@@ -128,11 +93,4 @@
         </geometry>
       </collision>
-      <inertial>
-          <mass value="0.568760"/>
-          <origin xyz="0.000000 0.049931 0.022823" rpy="0.0 0.0 0.0"/>
-          <inertia ixx="0.001084" ixy="0.000000" ixz="0.000000"
-                                  iyy="0.001123" iyz="0.000001"
-                                                 izz="0.000383"/>
-      </inertial>
     </link>
     <link name="${prefix}link_6">
@@ -150,11 +108,4 @@
         </geometry>
       </collision>
-      <inertial>
-          <mass value="0.030977"/>
-          <origin xyz="-0.000243 0.050000 -0.206293" rpy="0.0 0.0 0.0"/>
-          <inertia ixx="0.000012" ixy="-0.000000" ixz="0.000000"
-                                  iyy="0.000011"  iyz="0.000000"
-                                                  izz="0.000022"/>
-      </inertial>
     </link>
     <!-- joints: main serial chain -->

File: staubli_tx2_90_support/urdf/tx2_90xl_macro.xacro (robot description, xacro)
@@ -18,11 +18,4 @@
         </geometry>
       </collision>
-      <inertial>
-          <mass value="10.733459"/>
-          <origin xyz="0.014288 0.000001 0.122264" rpy="0.0 0.0 0.0"/>
-          <inertia ixx="0.096590" ixy="-0.000005" ixz="-0.003803"
-                                  iyy="0.087591"  iyz="-0.000001"
-                                                  izz="0.081632"/>
-      </inertial>
     </link>
     <link name="${prefix}link_1">
@@ -40,11 +33,4 @@
         </geometry>
       </collision>
-      <inertial>
-          <mass value="16.934564"/>
-          <origin xyz="0.019143 0.024764 -0.064596" rpy="0.0 0.0 0.0"/>
-          <inertia ixx="0.222318" ixy="0.016499" ixz="0.023794"
-                                  iyy="0.208959" iyz="0.031663"
-                                                 izz="0.157081"/>
-      </inertial>
     </link>
     <link name="${prefix}link_2">
@@ -62,11 +48,4 @@
         </geometry>
       </collision>
-      <inertial>
-          <mass value="14.350897"/>
-          <origin xyz="-0.000007 0.221192 0.206856" rpy="0.0 0.0 0.0"/>
-          <inertia ixx="0.595207" ixy="0.000005" ixz="-0.000008"
-                                  iyy="0.625683" iyz="-0.003766"
-                                                 izz="0.059863"/>
-      </inertial>
     </link>
     <link name="${prefix}link_3">
@@ -84,11 +63,4 @@
         </geometry>
       </collision>
-      <inertial>
-          <mass value="7.501506"/>
-          <origin xyz="0.000002 0.065008 -0.071428" rpy="0.0 0.0 0.0"/>
-          <inertia ixx="0.058902" ixy="0.000000" ixz="0.000001"
-                                  iyy="0.056884" iyz="-0.003672"
-                                                 izz="0.034271"/>
-      </inertial>
     </link>
     <link name="${prefix}link_4">
@@ -106,11 +78,4 @@
         </geometry>
       </collision>
-      <inertial>
-          <mass value="6.420429"/>
-          <origin xyz="-0.001998 0.049992 0.360301" rpy="0.0 0.0 0.0"/>
-          <inertia ixx="0.103999" ixy="0.000003" ixz="-0.001379"
-                                  iyy="0.098782" iyz="-0.000007"
-                                                 izz="0.019071"/>
-      </inertial>
     </link>
     <link name="${prefix}link_5">
@@ -128,11 +93,4 @@
         </geometry>
       </collision>
-      <inertial>
-          <mass value="0.568760"/>
-          <origin xyz="0.000000 0.049931 0.022823" rpy="0.0 0.0 0.0"/>
-          <inertia ixx="0.001084" ixy="0.000000" ixz="0.000000"
-                                  iyy="0.001123" iyz="0.000001"
-                                                 izz="0.000383"/>
-      </inertial>
     </link>
     <link name="${prefix}link_6">
@@ -150,11 +108,4 @@
         </geometry>
       </collision>
-      <inertial>
-          <mass value="0.030977"/>
-          <origin xyz="-0.000243 0.050000 -0.206293" rpy="0.0 0.0 0.0"/>
-          <inertia ixx="0.000012" ixy="-0.000000" ixz="0.000000"
-                                  iyy="0.000011"  iyz="0.000000"
-                                                  izz="0.000022"/>
-      </inertial>
     </link>
     <!-- joints: main serial chain -->

Commit message: rechecked limits with handbook and clarified reference

File: staubli_tx2_90_support/urdf/tx2_90_macro.xacro (robot description, xacro)
@@ -126,5 +126,5 @@
       <child link="${prefix}link_2"/>
       <axis xyz="0 1 0"/>
-      <limit lower="${radians(-130)}" upper="${radians(147.5)}" effort="130.0" velocity="${radians(390)}" />
+      <limit lower="${radians(-130)}" upper="${radians(147.5)}" effort="166.0" velocity="${radians(400)}" />
       <dynamics damping="0.0" friction="0.0"/>
     </joint>
@@ -134,5 +134,5 @@
       <child link="${prefix}link_3"/>
       <axis xyz="0 1 0"/>
-      <limit lower="${radians(-145)}" upper="${radians(145)}" effort="65.0" velocity="${radians(420)}" />
+      <limit lower="${radians(-145)}" upper="${radians(145)}" effort="76.0" velocity="${radians(430)}" />
       <dynamics damping="0.0" friction="0.0"/>
     </joint>

File: staubli_tx2_90_support/urdf/tx2_90xl_macro.xacro (robot description, xacro)
@@ -126,5 +126,5 @@
       <child link="${prefix}link_2"/>
       <axis xyz="0 1 0"/>
-      <limit lower="${radians(-130)}" upper="${radians(147.5)}" effort="130.0" velocity="${radians(390)}" />
+      <limit lower="${radians(-130)}" upper="${radians(147.5)}" effort="90.0" velocity="${radians(350)}" />
       <dynamics damping="0.0" friction="0.0"/>
     </joint>
@@ -134,5 +134,5 @@
       <child link="${prefix}link_3"/>
       <axis xyz="0 1 0"/>
-      <limit lower="${radians(-145)}" upper="${radians(145)}" effort="65.0" velocity="${radians(420)}" />
+      <limit lower="${radians(-145)}" upper="${radians(145)}" effort="53.0" velocity="${radians(410)}" />
       <dynamics damping="0.0" friction="0.0"/>
     </joint>

Commit message: use nominal speed limits

File: staubli_tx2_90_support/urdf/tx2_90_macro.xacro (robot description, xacro)
@@ -118,5 +118,6 @@
       (1) effort limit = 318 Nm if floor mounted
       (2) effort limit = 111 Nm if wall mounted -->
-      <limit lower="${radians(-180)}" upper="${radians(180)}" effort="318.0" velocity="${radians(400)}" />
+      <!-- nominal speed limits are used -->
+      <limit lower="${radians(-180)}" upper="${radians(180)}" effort="318.0" velocity="${radians(265)}" />
       <dynamics damping="0.0" friction="0.0"/>
     </joint>
@@ -126,5 +127,5 @@
       <child link="${prefix}link_2"/>
       <axis xyz="0 1 0"/>
-      <limit lower="${radians(-130)}" upper="${radians(147.5)}" effort="166.0" velocity="${radians(400)}" />
+      <limit lower="${radians(-130)}" upper="${radians(147.5)}" effort="166.0" velocity="${radians(210)}" />
       <dynamics damping="0.0" friction="0.0"/>
     </joint>
@@ -134,5 +135,5 @@
       <child link="${prefix}link_3"/>
       <axis xyz="0 1 0"/>
-      <limit lower="${radians(-145)}" upper="${radians(145)}" effort="76.0" velocity="${radians(430)}" />
+      <limit lower="${radians(-145)}" upper="${radians(145)}" effort="76.0" velocity="${radians(315)}" />
       <dynamics damping="0.0" friction="0.0"/>
     </joint>
@@ -142,5 +143,5 @@
       <child link="${prefix}link_4"/>
       <axis xyz="0 0 1"/>
-      <limit lower="${radians(-270)}" upper="${radians(270)}" effort="34.0" velocity="${radians(540)}" />
+      <limit lower="${radians(-270)}" upper="${radians(270)}" effort="34.0" velocity="${radians(450)}" />
       <dynamics damping="0.0" friction="0.0"/>
     </joint>
@@ -150,5 +151,5 @@
       <child link="${prefix}link_5"/>
       <axis xyz="0 1 0"/>
-      <limit lower="${radians(-115)}" upper="${radians(140)}" effort="29.0" velocity="${radians(475)}" />
+      <limit lower="${radians(-115)}" upper="${radians(140)}" effort="29.0" velocity="${radians(370)}" />
       <dynamics damping="0.0" friction="0.0"/>
     </joint>
@@ -158,5 +159,5 @@
       <child link="${prefix}link_6"/>
       <axis xyz="0 0 1"/>
-      <limit lower="${radians(-270)}" upper="${radians(270)}" effort="11.0" velocity="${radians(760)}" />
+      <limit lower="${radians(-270)}" upper="${radians(270)}" effort="11.0" velocity="${radians(630)}" />
       <dynamics damping="0.0" friction="0.0"/>
     </joint>

File: staubli_tx2_90_support/urdf/tx2_90l_macro.xacro (robot description, xacro)
@@ -118,5 +118,6 @@
       (1) effort limit = 318 Nm if floor mounted
       (2) effort limit = 111 Nm if wall mounted -->
-      <limit lower="${radians(-180)}" upper="${radians(180)}" effort="318.0" velocity="${radians(400)}" />
+      <!-- nominal speed limits are used -->
+      <limit lower="${radians(-180)}" upper="${radians(180)}" effort="318.0" velocity="${radians(225)}" />
       <dynamics damping="0.0" friction="0.0"/>
     </joint>
@@ -126,5 +127,5 @@
       <child link="${prefix}link_2"/>
       <axis xyz="0 1 0"/>
-      <limit lower="${radians(-130)}" upper="${radians(147.5)}" effort="130.0" velocity="${radians(390)}" />
+      <limit lower="${radians(-130)}" upper="${radians(147.5)}" effort="130.0" velocity="${radians(180)}" />
       <dynamics damping="0.0" friction="0.0"/>
     </joint>
@@ -134,5 +135,5 @@
       <child link="${prefix}link_3"/>
       <axis xyz="0 1 0"/>
-      <limit lower="${radians(-145)}" upper="${radians(145)}" effort="65.0" velocity="${radians(420)}" />
+      <limit lower="${radians(-145)}" upper="${radians(145)}" effort="65.0" velocity="${radians(270)}" />
       <dynamics damping="0.0" friction="0.0"/>
     </joint>
@@ -142,5 +143,5 @@
       <child link="${prefix}link_4"/>
       <axis xyz="0 0 1"/>
-      <limit lower="${radians(-270)}" upper="${radians(270)}" effort="34.0" velocity="${radians(540)}" />
+      <limit lower="${radians(-270)}" upper="${radians(270)}" effort="34.0" velocity="${radians(450)}" />
       <dynamics damping="0.0" friction="0.0"/>
     </joint>
@@ -150,5 +151,5 @@
       <child link="${prefix}link_5"/>
       <axis xyz="0 1 0"/>
-      <limit lower="${radians(-115)}" upper="${radians(140)}" effort="29.0" velocity="${radians(475)}" />
+      <limit lower="${radians(-115)}" upper="${radians(140)}" effort="29.0" velocity="${radians(370)}" />
       <dynamics damping="0.0" friction="0.0"/>
     </joint>
@@ -158,5 +159,5 @@
       <child link="${prefix}link_6"/>
       <axis xyz="0 0 1"/>
-      <limit lower="${radians(-270)}" upper="${radians(270)}" effort="11.0" velocity="${radians(760)}" />
+      <limit lower="${radians(-270)}" upper="${radians(270)}" effort="11.0" velocity="${radians(630)}" />
       <dynamics damping="0.0" friction="0.0"/>
     </joint>

File: staubli_tx2_90_support/urdf/tx2_90xl_macro.xacro (robot description, xacro)
@@ -118,5 +118,6 @@
       (1) effort limit = 318 Nm if floor mounted
       (2) effort limit = 111 Nm if wall mounted -->
-      <limit lower="${radians(-180)}" upper="${radians(180)}" effort="318.0" velocity="${radians(400)}" />
+      <!-- nominal speed limits are used -->
+      <limit lower="${radians(-180)}" upper="${radians(180)}" effort="318.0" velocity="${radians(200)}" />
       <dynamics damping="0.0" friction="0.0"/>
     </joint>
@@ -126,5 +127,5 @@
       <child link="${prefix}link_2"/>
       <axis xyz="0 1 0"/>
-      <limit lower="${radians(-130)}" upper="${radians(147.5)}" effort="90.0" velocity="${radians(350)}" />
+      <limit lower="${radians(-130)}" upper="${radians(147.5)}" effort="90.0" velocity="${radians(170)}" />
       <dynamics damping="0.0" friction="0.0"/>
     </joint>
@@ -134,5 +135,5 @@
       <child link="${prefix}link_3"/>
       <axis xyz="0 1 0"/>
-      <limit lower="${radians(-145)}" upper="${radians(145)}" effort="53.0" velocity="${radians(410)}" />
+      <limit lower="${radians(-145)}" upper="${radians(145)}" effort="53.0" velocity="${radians(240)}" />
       <dynamics damping="0.0" friction="0.0"/>
     </joint>
@@ -142,5 +143,5 @@
       <child link="${prefix}link_4"/>
       <axis xyz="0 0 1"/>
-      <limit lower="${radians(-270)}" upper="${radians(270)}" effort="34.0" velocity="${radians(540)}" />
+      <limit lower="${radians(-270)}" upper="${radians(270)}" effort="34.0" velocity="${radians(420)}" />
       <dynamics damping="0.0" friction="0.0"/>
     </joint>
@@ -150,5 +151,5 @@
       <child link="${prefix}link_5"/>
       <axis xyz="0 1 0"/>
-      <limit lower="${radians(-115)}" upper="${radians(140)}" effort="29.0" velocity="${radians(475)}" />
+      <limit lower="${radians(-115)}" upper="${radians(140)}" effort="29.0" velocity="${radians(360)}" />
       <dynamics damping="0.0" friction="0.0"/>
     </joint>
@@ -158,5 +159,5 @@
       <child link="${prefix}link_6"/>
       <axis xyz="0 0 1"/>
-      <limit lower="${radians(-270)}" upper="${radians(270)}" effort="11.0" velocity="${radians(760)}" />
+      <limit lower="${radians(-270)}" upper="${radians(270)}" effort="11.0" velocity="${radians(630)}" />
       <dynamics damping="0.0" friction="0.0"/>
     </joint>
