Commit message: Remove dynamics elements as well.
No use keeping them if inertial is not present.

File: staubli_tx2_90_support/urdf/tx2_90_macro.xacro (robot description, xacro)
@@ -120,5 +120,4 @@
       <!-- nominal velocity limits are used -->
       <limit lower="${radians(-180)}" upper="${radians(180)}" effort="318.0" velocity="${radians(265)}" />
-      <dynamics damping="0.0" friction="0.0"/>
     </joint>
     <joint name="${prefix}joint_2" type="revolute">
@@ -129,5 +128,4 @@
       <!-- nominal velocity limits are used -->
       <limit lower="${radians(-130)}" upper="${radians(147.5)}" effort="166.0" velocity="${radians(210)}" />
-      <dynamics damping="0.0" friction="0.0"/>
     </joint>
     <joint name="${prefix}joint_3" type="revolute">
@@ -138,5 +136,4 @@
       <!-- nominal velocity limits are used -->
       <limit lower="${radians(-145)}" upper="${radians(145)}" effort="76.0" velocity="${radians(315)}" />
-      <dynamics damping="0.0" friction="0.0"/>
     </joint>
     <joint name="${prefix}joint_4" type="revolute">
@@ -147,5 +144,4 @@
       <!-- nominal velocity limits are used -->
       <limit lower="${radians(-270)}" upper="${radians(270)}" effort="34.0" velocity="${radians(450)}" />
-      <dynamics damping="0.0" friction="0.0"/>
     </joint>
     <joint name="${prefix}joint_5" type="revolute">
@@ -156,5 +152,4 @@
       <!-- nominal velocity limits are used -->
       <limit lower="${radians(-115)}" upper="${radians(140)}" effort="29.0" velocity="${radians(370)}" />
-      <dynamics damping="0.0" friction="0.0"/>
     </joint>
     <joint name="${prefix}joint_6" type="revolute">
@@ -165,5 +160,4 @@
       <!-- nominal velocity limits are used -->
       <limit lower="${radians(-270)}" upper="${radians(270)}" effort="11.0" velocity="${radians(630)}" />
-      <dynamics damping="0.0" friction="0.0"/>
     </joint>
     <!-- ROS-Industrial 'base' frame: base_link to Staubli World Coordinates transform -->

File: staubli_tx2_90_support/urdf/tx2_90l_macro.xacro (robot description, xacro)
@@ -120,5 +120,4 @@
       <!-- nominal velocity limits are used -->
       <limit lower="${radians(-180)}" upper="${radians(180)}" effort="318.0" velocity="${radians(225)}" />
-      <dynamics damping="0.0" friction="0.0"/>
     </joint>
     <joint name="${prefix}joint_2" type="revolute">
@@ -129,5 +128,4 @@
       <!-- nominal velocity limits are used -->
       <limit lower="${radians(-130)}" upper="${radians(147.5)}" effort="130.0" velocity="${radians(180)}" />
-      <dynamics damping="0.0" friction="0.0"/>
     </joint>
     <joint name="${prefix}joint_3" type="revolute">
@@ -138,5 +136,4 @@
       <!-- nominal velocity limits are used -->
       <limit lower="${radians(-145)}" upper="${radians(145)}" effort="65.0" velocity="${radians(270)}" />
-      <dynamics damping="0.0" friction="0.0"/>
     </joint>
     <joint name="${prefix}joint_4" type="revolute">
@@ -147,5 +144,4 @@
       <!-- nominal velocity limits are used -->
       <limit lower="${radians(-270)}" upper="${radians(270)}" effort="34.0" velocity="${radians(450)}" />
-      <dynamics damping="0.0" friction="0.0"/>
     </joint>
     <joint name="${prefix}joint_5" type="revolute">
@@ -156,5 +152,4 @@
       <!-- nominal velocity limits are used -->
       <limit lower="${radians(-115)}" upper="${radians(140)}" effort="29.0" velocity="${radians(370)}" />
-      <dynamics damping="0.0" friction="0.0"/>
     </joint>
     <joint name="${prefix}joint_6" type="revolute">
@@ -165,5 +160,4 @@
       <!-- nominal velocity limits are used -->
       <limit lower="${radians(-270)}" upper="${radians(270)}" effort="11.0" velocity="${radians(630)}" />
-      <dynamics damping="0.0" friction="0.0"/>
     </joint>
     <!-- ROS-Industrial 'base' frame: base_link to Staubli World Coordinates transform -->

File: staubli_tx2_90_support/urdf/tx2_90xl_macro.xacro (robot description, xacro)
@@ -120,5 +120,4 @@
       <!-- nominal velocity limits are used -->
       <limit lower="${radians(-180)}" upper="${radians(180)}" effort="318.0" velocity="${radians(200)}" />
-      <dynamics damping="0.0" friction="0.0"/>
     </joint>
     <joint name="${prefix}joint_2" type="revolute">
@@ -129,5 +128,4 @@
       <!-- nominal velocity limits are used -->
       <limit lower="${radians(-130)}" upper="${radians(147.5)}" effort="90.0" velocity="${radians(170)}" />
-      <dynamics damping="0.0" friction="0.0"/>
     </joint>
     <joint name="${prefix}joint_3" type="revolute">
@@ -138,5 +136,4 @@
       <!-- nominal velocity limits are used -->
       <limit lower="${radians(-145)}" upper="${radians(145)}" effort="53.0" velocity="${radians(240)}" />
-      <dynamics damping="0.0" friction="0.0"/>
     </joint>
     <joint name="${prefix}joint_4" type="revolute">
@@ -147,5 +144,4 @@
       <!-- nominal velocity limits are used -->
       <limit lower="${radians(-270)}" upper="${radians(270)}" effort="34.0" velocity="${radians(420)}" />
-      <dynamics damping="0.0" friction="0.0"/>
     </joint>
     <joint name="${prefix}joint_5" type="revolute">
@@ -156,5 +152,4 @@
       <!-- nominal velocity limits are used -->
       <limit lower="${radians(-115)}" upper="${radians(140)}" effort="29.0" velocity="${radians(360)}" />
-      <dynamics damping="0.0" friction="0.0"/>
     </joint>
     <joint name="${prefix}joint_6" type="revolute">
@@ -165,5 +160,4 @@
       <!-- nominal velocity limits are used -->
       <limit lower="${radians(-270)}" upper="${radians(270)}" effort="11.0" velocity="${radians(630)}" />
-      <dynamics damping="0.0" friction="0.0"/>
     </joint>
     <!-- ROS-Industrial 'base' frame: base_link to Staubli World Coordinates transform -->

Commit message: Make flange parent of tool0.

File: staubli_tx2_90_support/urdf/tx2_90_macro.xacro (robot description, xacro)
@@ -177,8 +177,8 @@
     <!-- ROS-Industrial 'tool0' frame: all-zeros tool frame -->
     <link name="${prefix}tool0" />
-    <joint name="${prefix}joint_6-tool0" type="fixed">
-      <parent link="${prefix}link_6"/>
-      <child link="${prefix}tool0"/>
-      <origin xyz="0 0 0" rpy="0 0 0"/>
+    <joint name="${prefix}flange-tool0" type="fixed">
+      <parent link="${prefix}flange" />
+      <child link="${prefix}tool0" />
+      <origin xyz="0 0 0" rpy="0 ${radians(90.0)} 0" />
     </joint>
   </xacro:macro>

File: staubli_tx2_90_support/urdf/tx2_90l_macro.xacro (robot description, xacro)
@@ -177,8 +177,8 @@
     <!-- ROS-Industrial 'tool0' frame: all-zeros tool frame -->
     <link name="${prefix}tool0" />
-        <joint name="${prefix}joint_6-tool0" type="fixed">
-      <parent link="${prefix}link_6"/>
-      <child link="${prefix}tool0"/>
-      <origin xyz="0 0 0" rpy="0 0 0"/>
+    <joint name="${prefix}flange-tool0" type="fixed">
+      <parent link="${prefix}flange" />
+      <child link="${prefix}tool0" />
+      <origin xyz="0 0 0" rpy="0 ${radians(90.0)} 0" />
     </joint>
   </xacro:macro>

File: staubli_tx2_90_support/urdf/tx2_90xl_macro.xacro (robot description, xacro)
@@ -177,8 +177,8 @@
     <!-- ROS-Industrial 'tool0' frame: all-zeros tool frame -->
     <link name="${prefix}tool0" />
-    <joint name="${prefix}joint_6-tool0" type="fixed">
-      <parent link="${prefix}link_6"/>
-      <child link="${prefix}tool0"/>
-      <origin xyz="0 0 0" rpy="0 0 0"/>
+    <joint name="${prefix}flange-tool0" type="fixed">
+      <parent link="${prefix}flange" />
+      <child link="${prefix}tool0" />
+      <origin xyz="0 0 0" rpy="0 ${radians(90.0)} 0" />
     </joint>
   </xacro:macro>
