Commit message: change tx260 to tx2_60

File: staubli_tx2_60_support/urdf/tx2_60_macro.xacro (robot description, xacro)
@@ -2,5 +2,5 @@
 <robot xmlns:xacro="http://wiki.ros.org/xacro">
   <xacro:include filename="$(find staubli_resources)/urdf/common_materials.xacro"/>
-  <xacro:macro name="staubli_tx260" params="prefix">
+  <xacro:macro name="staubli_tx2_60" params="prefix">
     <!-- links: main serial chain -->
     <link name="${prefix}base_link">
@@ -8,12 +8,12 @@
         <origin xyz="0 0 0" rpy="0 0 0"/>
         <geometry>
-          <mesh filename="package://staubli_tx260_support/meshes/tx260/visual/base_link.stl"/>
-        </geometry>
-        <xacro:material_staubli_ral_melon_yellow />
-      </visual>
-      <collision>
-        <origin xyz="0 0 0" rpy="0 0 0"/>
-        <geometry>
-          <mesh filename="package://staubli_tx260_support/meshes/tx260/collision/base_link.stl"/>
+          <mesh filename="package://staubli_tx2_60_support/meshes/tx2_60/visual/base_link.stl"/>
+        </geometry>
+        <xacro:material_staubli_ral_melon_yellow />
+      </visual>
+      <collision>
+        <origin xyz="0 0 0" rpy="0 0 0"/>
+        <geometry>
+          <mesh filename="package://staubli_tx2_60_support/meshes/tx2_60/collision/base_link.stl"/>
         </geometry>
       </collision>
@@ -30,12 +30,12 @@
         <origin xyz="0 0 0" rpy="0 0 0"/>
         <geometry>
-          <mesh filename="package://staubli_tx260_support/meshes/tx260/visual/link_1.stl"/>
-        </geometry>
-        <xacro:material_staubli_ral_melon_yellow />
-      </visual>
-      <collision>
-        <origin xyz="0 0 0" rpy="0 0 0"/>
-        <geometry>
-          <mesh filename="package://staubli_tx260_support/meshes/tx260/collision/link_1.stl"/>
+          <mesh filename="package://staubli_tx2_60_support/meshes/tx2_60/visual/link_1.stl"/>
+        </geometry>
+        <xacro:material_staubli_ral_melon_yellow />
+      </visual>
+      <collision>
+        <origin xyz="0 0 0" rpy="0 0 0"/>
+        <geometry>
+          <mesh filename="package://staubli_tx2_60_support/meshes/tx2_60/collision/link_1.stl"/>
         </geometry>
       </collision>
@@ -52,12 +52,12 @@
         <origin xyz="0 0 0" rpy="0 0 0"/>
         <geometry>
-          <mesh filename="package://staubli_tx260_support/meshes/tx260/visual/link_2.stl"/>
-        </geometry>
-        <xacro:material_staubli_ral_melon_yellow />
-      </visual>
-      <collision>
-        <origin xyz="0 0 0" rpy="0 0 0"/>
-        <geometry>
-          <mesh filename="package://staubli_tx260_support/meshes/tx260/collision/link_2.stl"/>
+          <mesh filename="package://staubli_tx2_60_support/meshes/tx2_60/visual/link_2.stl"/>
+        </geometry>
+        <xacro:material_staubli_ral_melon_yellow />
+      </visual>
+      <collision>
+        <origin xyz="0 0 0" rpy="0 0 0"/>
+        <geometry>
+          <mesh filename="package://staubli_tx2_60_support/meshes/tx2_60/collision/link_2.stl"/>
         </geometry>
       </collision>
@@ -74,12 +74,12 @@
         <origin xyz="0 0 0" rpy="0 0 0"/>
         <geometry>
-          <mesh filename="package://staubli_tx260_support/meshes/tx260/visual/link_3.stl"/>
-        </geometry>
-        <xacro:material_staubli_ral_melon_yellow />
-      </visual>
-      <collision>
-        <origin xyz="0 0 0" rpy="0 0 0"/>
-        <geometry>
-          <mesh filename="package://staubli_tx260_support/meshes/tx260/collision/link_3.stl"/>
+          <mesh filename="package://staubli_tx2_60_support/meshes/tx2_60/visual/link_3.stl"/>
+        </geometry>
+        <xacro:material_staubli_ral_melon_yellow />
+      </visual>
+      <collision>
+        <origin xyz="0 0 0" rpy="0 0 0"/>
+        <geometry>
+          <mesh filename="package://staubli_tx2_60_support/meshes/tx2_60/collision/link_3.stl"/>
         </geometry>
       </collision>
@@ -96,12 +96,12 @@
         <origin xyz="0 0 0" rpy="0 0 0"/>
         <geometry>
-          <mesh filename="package://staubli_tx260_support/meshes/tx260/visual/link_4.stl"/>
-        </geometry>
-        <xacro:material_staubli_ral_melon_yellow />
-      </visual>
-      <collision>
-        <origin xyz="0 0 0" rpy="0 0 0"/>
-        <geometry>
-          <mesh filename="package://staubli_tx260_support/meshes/tx260/collision/link_4.stl"/>
+          <mesh filename="package://staubli_tx2_60_support/meshes/tx2_60/visual/link_4.stl"/>
+        </geometry>
+        <xacro:material_staubli_ral_melon_yellow />
+      </visual>
+      <collision>
+        <origin xyz="0 0 0" rpy="0 0 0"/>
+        <geometry>
+          <mesh filename="package://staubli_tx2_60_support/meshes/tx2_60/collision/link_4.stl"/>
         </geometry>
       </collision>

File: staubli_tx2_60_support/urdf/tx2_60l_macro.xacro (robot description, xacro)
@@ -2,5 +2,5 @@
 <robot xmlns:xacro="http://wiki.ros.org/xacro">
   <xacro:include filename="$(find staubli_resources)/urdf/common_materials.xacro"/>
-  <xacro:macro name="staubli_tx260l" params="prefix">
+  <xacro:macro name="staubli_tx2_60l" params="prefix">
     <!-- links: main serial chain -->
     <link name="${prefix}base_link">
@@ -8,12 +8,12 @@
         <origin xyz="0 0 0" rpy="0 0 0"/>
         <geometry>
-          <mesh filename="package://staubli_tx260_support/meshes/tx260/visual/base_link.stl"/>
-        </geometry>
-        <xacro:material_staubli_ral_melon_yellow />
-      </visual>
-      <collision>
-        <origin xyz="0 0 0" rpy="0 0 0"/>
-        <geometry>
-          <mesh filename="package://staubli_tx260_support/meshes/tx260/collision/base_link.stl"/>
+          <mesh filename="package://staubli_tx2_60_support/meshes/tx2_60/visual/base_link.stl"/>
+        </geometry>
+        <xacro:material_staubli_ral_melon_yellow />
+      </visual>
+      <collision>
+        <origin xyz="0 0 0" rpy="0 0 0"/>
+        <geometry>
+          <mesh filename="package://staubli_tx2_60_support/meshes/tx2_60/collision/base_link.stl"/>
         </geometry>
       </collision>
@@ -30,12 +30,12 @@
         <origin xyz="0 0 0" rpy="0 0 0"/>
         <geometry>
-          <mesh filename="package://staubli_tx260_support/meshes/tx260/visual/link_1.stl"/>
-        </geometry>
-        <xacro:material_staubli_ral_melon_yellow />
-      </visual>
-      <collision>
-        <origin xyz="0 0 0" rpy="0 0 0"/>
-        <geometry>
-          <mesh filename="package://staubli_tx260_support/meshes/tx260/collision/link_1.stl"/>
+          <mesh filename="package://staubli_tx2_60_support/meshes/tx2_60/visual/link_1.stl"/>
+        </geometry>
+        <xacro:material_staubli_ral_melon_yellow />
+      </visual>
+      <collision>
+        <origin xyz="0 0 0" rpy="0 0 0"/>
+        <geometry>
+          <mesh filename="package://staubli_tx2_60_support/meshes/tx2_60/collision/link_1.stl"/>
         </geometry>
       </collision>
@@ -52,12 +52,12 @@
         <origin xyz="0 0 0" rpy="0 0 0"/>
         <geometry>
-          <mesh filename="package://staubli_tx260_support/meshes/tx260l/visual/link_2.stl"/>
-        </geometry>
-        <xacro:material_staubli_ral_melon_yellow />
-      </visual>
-      <collision>
-        <origin xyz="0 0 0" rpy="0 0 0"/>
-        <geometry>
-          <mesh filename="package://staubli_tx260_support/meshes/tx260l/collision/link_2.stl"/>
+          <mesh filename="package://staubli_tx2_60_support/meshes/tx2_60l/visual/link_2.stl"/>
+        </geometry>
+        <xacro:material_staubli_ral_melon_yellow />
+      </visual>
+      <collision>
+        <origin xyz="0 0 0" rpy="0 0 0"/>
+        <geometry>
+          <mesh filename="package://staubli_tx2_60_support/meshes/tx2_60l/collision/link_2.stl"/>
         </geometry>
       </collision>
@@ -74,12 +74,12 @@
         <origin xyz="0 0 0" rpy="0 0 0"/>
         <geometry>
-          <mesh filename="package://staubli_tx260_support/meshes/tx260/visual/link_3.stl"/>
-        </geometry>
-        <xacro:material_staubli_ral_melon_yellow />
-      </visual>
-      <collision>
-        <origin xyz="0 0 0" rpy="0 0 0"/>
-        <geometry>
-          <mesh filename="package://staubli_tx260_support/meshes/tx260/collision/link_3.stl"/>
+          <mesh filename="package://staubli_tx2_60_support/meshes/tx2_60/visual/link_3.stl"/>
+        </geometry>
+        <xacro:material_staubli_ral_melon_yellow />
+      </visual>
+      <collision>
+        <origin xyz="0 0 0" rpy="0 0 0"/>
+        <geometry>
+          <mesh filename="package://staubli_tx2_60_support/meshes/tx2_60/collision/link_3.stl"/>
         </geometry>
       </collision>
@@ -96,12 +96,12 @@
         <origin xyz="0 0 0" rpy="0 0 0"/>
         <geometry>
-          <mesh filename="package://staubli_tx260_support/meshes/tx260l/visual/link_4.stl"/>
-        </geometry>
-        <xacro:material_staubli_ral_melon_yellow />
-      </visual>
-      <collision>
-        <origin xyz="0 0 0" rpy="0 0 0"/>
-        <geometry>
-          <mesh filename="package://staubli_tx260_support/meshes/tx260l/collision/link_4.stl"/>
+          <mesh filename="package://staubli_tx2_60_support/meshes/tx2_60l/visual/link_4.stl"/>
+        </geometry>
+        <xacro:material_staubli_ral_melon_yellow />
+      </visual>
+      <collision>
+        <origin xyz="0 0 0" rpy="0 0 0"/>
+        <geometry>
+          <mesh filename="package://staubli_tx2_60_support/meshes/tx2_60l/collision/link_4.stl"/>
         </geometry>
       </collision>

Commit message: removing inertial from xacros

File: staubli_tx2_60_support/urdf/tx2_60_macro.xacro (robot description, xacro)
@@ -18,11 +18,4 @@
         </geometry>
       </collision>
-      <inertial>
-          <mass value="4.65971957"/>
-          <origin xyz="-0.00257355 -0.00039402 0.08786146" rpy="0.0 0.0 0.0"/>
-          <inertia ixx="0.02319781" ixy="0.00023234" ixz="0.00162421"
-                                    iyy="0.02621322" iyz="0.00008092"
-                                                     izz="0.02286303"/>
-      </inertial>
     </link>
     <link name="${prefix}link_1">
@@ -40,11 +33,4 @@
         </geometry>
       </collision>
-      <inertial>
-          <mass value="6.99103376"/>
-          <origin xyz="0.00000000 0.02467680 -0.05265925" rpy="0.0 0.0 0.0"/>
-          <inertia ixx="0.05672953" ixy="0.00000037" ixz="-0.00000049"
-                                    iyy="0.04909238" iyz="0.01016069"
-                                                     izz="0.03457565"/>
-      </inertial>
     </link>
     <link name="${prefix}link_2">
@@ -62,11 +48,4 @@
         </geometry>
       </collision>
-      <inertial>
-          <mass value="5.21353000"/>
-          <origin xyz="-0.00000322 0.17137541 0.17514843" rpy="0.0 0.0 0.0"/>
-          <inertia ixx="0.13669961" ixy="0.00000038" ixz="-0.00000068"
-                                    iyy="0.14393633" iyz="-0.00049262"
-                                                     izz="0.01130291"/>
-      </inertial>
     </link>
     <link name="${prefix}link_3">
@@ -84,11 +63,4 @@
         </geometry>
       </collision>
-      <inertial>
-          <mass value="4.52768000"/>
-          <origin xyz="0.00424668 0.02553862 -0.00735408" rpy="0.0 0.0 0.0"/>
-          <inertia ixx="0.02469218" ixy="0.00032528" ixz="0.00063194"
-                                    iyy="0.02222651" iyz="-0.00155762"
-                                                     izz="0.01657366"/>
-      </inertial>
     </link>
     <link name="${prefix}link_4">
@@ -106,11 +78,4 @@
         </geometry>
       </collision>
-      <inertial>
-          <mass value="3.48055000"/>
-          <origin xyz="-0.00134244 -0.00000186 0.28816464" rpy="0.0 0.0 0.0"/>
-          <inertia ixx="0.03950054" ixy="0.00000004" ixz="-0.00063419"
-                                    iyy="0.03813828" iyz="-0.00000002"
-                                                     izz="0.00610289"/>
-      </inertial>
     </link>
     <link name="${prefix}link_5">
@@ -128,11 +93,4 @@
         </geometry>
       </collision>
-      <inertial>
-          <mass value="0.16254714"/>
-          <origin xyz="-0.00000105 0.00000000 0.01268974" rpy="0.0 0.0 0.0"/>
-          <inertia ixx="0.00012557" ixy="0.00000000" ixz="0.00000000"
-                                    iyy="0.00013289" iyz="0.00000000"
-                                                     izz="0.00006342"/>
-      </inertial>
     </link>
     <link name="${prefix}link_6">
@@ -150,11 +108,4 @@
         </geometry>
       </collision>
-      <inertial>
-          <mass value="0.00820000"/>
-          <origin xyz="-0.00022629 0.00000000 -0.00597808" rpy="0.0 0.0 0.0"/>
-          <inertia ixx="0.00000096" ixy="0.00000000" ixz="0.00000000"
-                                    iyy="0.00000093" iyz="0.00000000"
-                                                     izz="0.00000154"/>
-      </inertial>
     </link>
     <!-- joints: main serial chain -->

File: staubli_tx2_60_support/urdf/tx2_60l_macro.xacro (robot description, xacro)
@@ -18,11 +18,4 @@
         </geometry>
       </collision>
-      <inertial>
-          <mass value="4.65971957"/>
-          <origin xyz="-0.00257355 -0.00039402 0.08786146" rpy="0.0 0.0 0.0"/>
-          <inertia ixx="0.02319781" ixy="0.00023234" ixz="0.00162421"
-                                    iyy="0.02621322" iyz="0.00008092"
-                                                     izz="0.02286303"/>
-      </inertial>
     </link>
     <link name="${prefix}link_1">
@@ -40,11 +33,4 @@
         </geometry>
       </collision>
-      <inertial>
-          <mass value="6.99103376"/>
-          <origin xyz="0.00000000 0.02467680 -0.05265925" rpy="0.0 0.0 0.0"/>
-          <inertia ixx="0.05672953" ixy="0.00000037" ixz="-0.00000049"
-                                    iyy="0.04909238" iyz="0.01016069"
-                                                     izz="0.03457565"/>
-      </inertial>
     </link>
     <link name="${prefix}link_2">
@@ -62,11 +48,4 @@
         </geometry>
       </collision>
-      <inertial>
-          <mass value="5.21353000"/>
-          <origin xyz="-0.00000322 0.17137541 0.17514843" rpy="0.0 0.0 0.0"/>
-          <inertia ixx="0.13669961" ixy="0.00000038" ixz="-0.00000068"
-                                    iyy="0.14393633" iyz="-0.00049262"
-                                                     izz="0.01130291"/>
-      </inertial>
     </link>
     <link name="${prefix}link_3">
@@ -84,11 +63,4 @@
         </geometry>
       </collision>
-      <inertial>
-          <mass value="4.52768000"/>
-          <origin xyz="0.00424668 0.02553862 -0.00735408" rpy="0.0 0.0 0.0"/>
-          <inertia ixx="0.02469218" ixy="0.00032528" ixz="0.00063194"
-                                    iyy="0.02222651" iyz="-0.00155762"
-                                                     izz="0.01657366"/>
-      </inertial>
     </link>
     <link name="${prefix}link_4">
@@ -106,11 +78,4 @@
         </geometry>
       </collision>
-      <inertial>
-          <mass value="3.48055000"/>
-          <origin xyz="-0.00134244 -0.00000186 0.28816464" rpy="0.0 0.0 0.0"/>
-          <inertia ixx="0.03950054" ixy="0.00000004" ixz="-0.00063419"
-                                    iyy="0.03813828" iyz="-0.00000002"
-                                                     izz="0.00610289"/>
-      </inertial>
     </link>
     <link name="${prefix}link_5">
@@ -128,11 +93,4 @@
         </geometry>
       </collision>
-      <inertial>
-          <mass value="0.16254714"/>
-          <origin xyz="-0.00000105 0.00000000 0.01268974" rpy="0.0 0.0 0.0"/>
-          <inertia ixx="0.00012557" ixy="0.00000000" ixz="0.00000000"
-                                    iyy="0.00013289" iyz="0.00000000"
-                                                     izz="0.00006342"/>
-      </inertial>
     </link>
     <link name="${prefix}link_6">
@@ -150,11 +108,4 @@
         </geometry>
       </collision>
-      <inertial>
-          <mass value="0.00820000"/>
-          <origin xyz="-0.00022629 0.00000000 -0.00597808" rpy="0.0 0.0 0.0"/>
-          <inertia ixx="0.00000096" ixy="0.00000000" ixz="0.00000000"
-                                    iyy="0.00000093" iyz="0.00000000"
-                                                     izz="0.00000154"/>
-      </inertial>
     </link>
     <!-- joints: main serial chain -->

Commit message: Remove dynamics elements as well.
No use keeping them if inertial is not present.

File: staubli_tx2_60_support/urdf/tx2_60_macro.xacro (robot description, xacro)
@@ -119,5 +119,4 @@
       (2) effort limit = 40 Nm if wall mounted -->
       <limit lower="${radians(-180)}" upper="${radians(180)}" effort="126.0" velocity="${radians(435)}" />
-      <dynamics damping="0.0" friction="0.0"/>
     </joint>
     <joint name="${prefix}joint_2" type="revolute">
@@ -127,5 +126,4 @@
       <axis xyz="0 1 0"/>
       <limit lower="${radians(-127.5)}" upper="${radians(127.5)}" effort="47.0" velocity="${radians(385)}" />
-      <dynamics damping="0.0" friction="0.0"/>
     </joint>
     <joint name="${prefix}joint_3" type="revolute">
@@ -135,5 +133,4 @@
       <axis xyz="0 1 0"/>
       <limit lower="${radians(-152.5)}" upper="${radians(152.5)}" effort="32.0" velocity="${radians(500)}" />
-      <dynamics damping="0.0" friction="0.0"/>
     </joint>
     <joint name="${prefix}joint_4" type="revolute">
@@ -143,5 +140,4 @@
       <axis xyz="0 0 1"/>
       <limit lower="${radians(-270.0)}" upper="${radians(270.0)}" effort="7.0" velocity="${radians(995)}" />
-      <dynamics damping="0.0" friction="0.0"/>
     </joint>
     <joint name="${prefix}joint_5" type="revolute">
@@ -151,5 +147,4 @@
       <axis xyz="0 1 0"/>
       <limit lower="${radians(-121.0)}" upper="${radians(132.5)}" effort="8.0" velocity="${radians(1065)}" />
-      <dynamics damping="0.0" friction="0.0"/>
     </joint>
     <joint name="${prefix}joint_6" type="revolute">
@@ -159,5 +154,4 @@
       <axis xyz="0 0 1"/>
       <limit lower="${radians(-270.0)}" upper="${radians(270.0)}" effort="2.0" velocity="${radians(1445)}" />
-      <dynamics damping="0.0" friction="0.0"/>
     </joint>
     <!-- ROS-Industrial 'base' frame: base_link to Staubli World Coordinates transform -->

File: staubli_tx2_60_support/urdf/tx2_60l_macro.xacro (robot description, xacro)
@@ -119,5 +119,4 @@
       (2) effort limit = 40 Nm if wall mounted -->
       <limit lower="${radians(-180)}" upper="${radians(180)}" effort="126.0" velocity="${radians(435)}" />
-      <dynamics damping="0.0" friction="0.0"/>
     </joint>
     <joint name="${prefix}joint_2" type="revolute">
@@ -127,5 +126,4 @@
       <axis xyz="0 1 0"/>
       <limit lower="${radians(-127.5)}" upper="${radians(127.5)}" effort="47.0" velocity="${radians(385)}" />
-      <dynamics damping="0.0" friction="0.0"/>
     </joint>
     <joint name="${prefix}joint_3" type="revolute">
@@ -135,5 +133,4 @@
       <axis xyz="0 1 0"/>
       <limit lower="${radians(-152.5)}" upper="${radians(152.5)}" effort="32.0" velocity="${radians(500)}" />
-      <dynamics damping="0.0" friction="0.0"/>
     </joint>
     <joint name="${prefix}joint_4" type="revolute">
@@ -143,5 +140,4 @@
       <axis xyz="0 0 1"/>
       <limit lower="${radians(-270.0)}" upper="${radians(270.0)}" effort="7.0" velocity="${radians(995)}" />
-      <dynamics damping="0.0" friction="0.0"/>
     </joint>
     <joint name="${prefix}joint_5" type="revolute">
@@ -151,5 +147,4 @@
       <axis xyz="0 1 0"/>
       <limit lower="${radians(-121.0)}" upper="${radians(132.5)}" effort="8.0" velocity="${radians(1065)}" />
-      <dynamics damping="0.0" friction="0.0"/>
     </joint>
     <joint name="${prefix}joint_6" type="revolute">
@@ -159,5 +154,4 @@
       <axis xyz="0 0 1"/>
       <limit lower="${radians(-270.0)}" upper="${radians(270.0)}" effort="2.0" velocity="${radians(1445)}" />
-      <dynamics damping="0.0" friction="0.0"/>
     </joint>
     <!-- ROS-Industrial 'base' frame: base_link to Staubli World Coordinates transform -->
