Commit message: tx2-60: apply suggested changes in PR for tx2-60 gazebo support

File: staubli_tx2_60_gazebo/urdf/tx2_60.xacro (robot description, xacro)
@@ -9,5 +9,5 @@
     <parent link="world"/>
     <child link="base_link"/>
-    <origin xyz="0.0 0.0 0.0" rpy="0.0 0.0 0.0" />
+    <origin xyz="0 0 0" rpy="0 0 0" />
   </joint>
 </robot>
